File: INPUT.sch (KiCad schematic (older format))
At the start: 42 parts

Commit message: current version of the schematics. Audio circuits are still missing.
Audio curcuit topology
Audio from cellphone module is routed to STM
Audio from microphone is routed to STM
STM processes audio and routes microphone data to cellphone module
STM processes audio and routes cellphone audio to amplifier
analog multiplexer can switch route from mic directly to cellphone module and module to speaker
Parts:
- removed Q? (x6): BC817-40, SOT-23, symbol BC817-40
- removed R? (x6): 1k, symbol R
- R701: renamed from R?; value R -> 10k
- SW701, SW702, SW703, SW704, SW705, SW706, SW707, SW708, SW709, SW710, SW711, SW712, SW713, SW714, SW715, SW716, SW717: renamed from SW?; footprint (none) -> buttons:Foil_Button
- gave numbers to parts that had none: 12
Connections:
- wire segments 82 -> 99
Other:
- moved on the sheet: R702, R704, R706, R708, R710, R712, SW702, SW703, SW704, SW705, SW706, SW707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

Commit message: added Ti WL1807/1837 Module for WLAN and Bluetooth. added Test Points
Parts:
- added TP? (x15): TP, symbol TP
Connections:
- wire segments 99 -> 63

Commit message: moved to some Bus routing for serveral communication signals on the top sheet. This reduces lines on the top sheet.
Changed 4V boost converter circuit toi use TPS61046 for size reasons
Connections:
- net labels added: KEY0, KEY1, KEY2, KEY3, KEY4, KEY5, KEY6, KEY7, KEY[0..7], LED0, LED1, LED2, LED3, LED4, LED5, LED[0..5]
- net labels removed: COL_1, COL_2, COL_3, COL_4, LED_1, LED_2, LED_3, LED_4, LED_5, LED_6, ROW_1, ROW_2, ROW_3, ROW_4
Other:
- moved on the sheet: TP?
Changed lines of the file:
@@
 LIBS:tp
 LIBS:w3006
+LIBS:tps61046
 LIBS:3210retro-cache
 EELAYER 25 0
@@
 $Descr A4 11693 8268
 encoding utf-8
-Sheet 5 9
+Sheet 7 9
 Title "Nokia 3210 Retrofit"
-Date "2016-12-20"
+Date "2016-12-22"
 Rev "1"
 Comp "www.kurzschluss-blog.de"
@@
 	1    0    0    -1
 $EndComp
-Text HLabel 2450 2450 1    60   Input ~ 0
-COL_1
-Text HLabel 3000 2450 1    60   Input ~ 0
-COL_2
-Text HLabel 3550 2450 1    60   Input ~ 0
-COL_3
-Text HLabel 4750 3150 2    60   Output ~ 0
-ROW_1
-Text HLabel 4750 4350 2    60   Output ~ 0
-ROW_3
-Text HLabel 4750 4950 2    60   Output ~ 0
-ROW_4
-Text HLabel 4750 3750 2    60   Output ~ 0
-ROW_2
-Text HLabel 4100 2450 1    60   Input ~ 0
-COL_4
 $Comp
 L GND #PWR502
@@
 	3250 3100 3300 3150
 Wire Wire Line
-	2750 3150 4750 3150
+	2750 3150 5000 3150
 Wire Wire Line
 	3850 3150 3800 3100
@@
 Connection ~ 4400 3150
 Wire Wire Line
-	2750 3750 4750 3750
+	2750 3750 5000 3750
 Wire Wire Line
 	4400 3750 4350 3700
@@
 	4100 3450 4150 3500
 Wire Wire Line
-	4100 2450 4100 4650
+	4100 2350 4100 4650
 Wire Wire Line
 	4100 2850 4150 2900
@@
 	3550 3450 3600 3500
 Wire Wire Line
-	3550 2450 3550 4650
+	3550 2350 3550 4650
 Wire Wire Line
 	3550 2850 3600 2900
@@
 	3000 3450 3050 3500
 Wire Wire Line
-	3000 2450 3000 4650
+	3000 2350 3000 4650
 Wire Wire Line
 	2450 3450 2500 3500
 Wire Wire Line
-	2450 2450 2450 4650
+	2450 2350 2450 4650
 Connection ~ 2450 2850
 Connection ~ 3000 2850
@@
 	2700 4300 2750 4350
 Wire Wire Line
-	2750 4350 4750 4350
+	2750 4350 5000 4350
 Wire Wire Line
 	3300 4350 3250 4300
@@
 	2700 4900 2750 4950
 Wire Wire Line
-	2750 4950 4750 4950
+	2750 4950 5000 4950
 Wire Wire Line
 	3300 4950 3250 4900
@@
 Wire Wire Line
 	9800 2800 9800 3000
-Wire Wire Line
-	7050 3400 7050 4100
 $Comp
 L +3V3 #PWR503
@@
 	9800 2400 9800 2500
 Connection ~ 9250 2400
-Text HLabel 7050 4100 3    60   Input ~ 0
-LED_1
-Text HLabel 7600 4100 3    60   Input ~ 0
-LED_2
-Wire Wire Line
-	7600 3400 7600 4100
-Text HLabel 8150 4100 3    60   Input ~ 0
-LED_3
-Wire Wire Line
-	8150 3400 8150 4100
-Text HLabel 8700 4100 3    60   Input ~ 0
-LED_4
-Wire Wire Line
-	8700 3400 8700 4100
-Text HLabel 9250 4100 3    60   Input ~ 0
-LED_5
-Wire Wire Line
-	9250 3400 9250 4100
-Text HLabel 9800 4100 3    60   Input ~ 0
-LED_6
-Wire Wire Line
-	9800 3400 9800 4100
+Wire Wire Line
+	7600 3400 7600 4700
+Wire Wire Line
+	8150 3400 8150 4700
+Wire Wire Line
+	8700 3400 8700 4700
+Wire Wire Line
+	9250 3400 9250 4700
+Wire Wire Line
+	9800 3400 9800 4700
 $Comp
 L TP TP?
@@
 L TP TP?
 U 1 1 585B7582
-P 2450 2650
-F 0 "TP?" H 2450 2690 20  0000 C CNN
-F 1 "TP" H 2450 2600 60  0001 C CNN
-F 2 "" H 2450 2650 60  0000 C CNN
-F 3 "" H 2450 2650 60  0000 C CNN
-	1    2450 2650
+P 2450 2750
+F 0 "TP?" H 2450 2790 20  0000 C CNN
+F 1 "TP" H 2450 2700 60  0001 C CNN
+F 2 "" H 2450 2750 60  0000 C CNN
+F 3 "" H 2450 2750 60  0000 C CNN
+	1    2450 2750
 	1    0    0    -1
 $EndComp
@@
 L TP TP?
 U 1 1 585B75E1
-P 3000 2650
-F 0 "TP?" H 3000 2690 20  0000 C CNN
-F 1 "TP" H 3000 2600 60  0001 C CNN
-F 2 "" H 3000 2650 60  0000 C CNN
-F 3 "" H 3000 2650 60  0000 C CNN
-	1    3000 2650
+P 3000 2750
+F 0 "TP?" H 3000 2790 20  0000 C CNN
+F 1 "TP" H 3000 2700 60  0001 C CNN
+F 2 "" H 3000 2750 60  0000 C CNN
+F 3 "" H 3000 2750 60  0000 C CNN
+	1    3000 2750
 	1    0    0    -1
 $EndComp
@@
 L TP TP?
 U 1 1 585B7642
-P 3550 2650
-F 0 "TP?" H 3550 2690 20  0000 C CNN
-F 1 "TP" H 3550 2600 60  0001 C CNN
-F 2 "" H 3550 2650 60  0000 C CNN
-F 3 "" H 3550 2650 60  0000 C CNN
-	1    3550 2650
+P 3550 2750
+F 0 "TP?" H 3550 2790 20  0000 C CNN
+F 1 "TP" H 3550 2700 60  0001 C CNN
+F 2 "" H 3550 2750 60  0000 C CNN
+F 3 "" H 3550 2750 60  0000 C CNN
+	1    3550 2750
 	1    0    0    -1
 $EndComp
@@
 L TP TP?
 U 1 1 585B7879
-P 4100 2650
-F 0 "TP?" H 4100 2690 20  0000 C CNN
-F 1 "TP" H 4100 2600 60  0001 C CNN
-F 2 "" H 4100 2650 60  0000 C CNN
-F 3 "" H 4100 2650 60  0000 C CNN
-	1    4100 2650
+P 4100 2750
+F 0 "TP?" H 4100 2790 20  0000 C CNN
+F 1 "TP" H 4100 2700 60  0001 C CNN
+F 2 "" H 4100 2750 60  0000 C CNN
+F 3 "" H 4100 2750 60  0000 C CNN
+	1    4100 2750
 	1    0    0    -1
 $EndComp
@@
 	1    0    0    -1
 $EndComp
+Wire Bus Line
+	1300 2250 5100 2250
+Entry Wire Line
+	2350 2250 2450 2350
+Entry Wire Line
+	2900 2250 3000 2350
+Entry Wire Line
+	3450 2250 3550 2350
+Entry Wire Line
+	4000 2250 4100 2350
+Entry Wire Line
+	5000 4950 5100 4850
+Entry Wire Line
+	5000 4350 5100 4250
+Entry Wire Line
+	5000 3750 5100 3650
+Entry Wire Line
+	5000 3150 5100 3050
+Text HLabel 1300 2250 0    60   BiDi ~ 0
+KEY[0..7]
+Wire Bus Line
+	5100 2250 5100 4850
+Text HLabel 6800 4800 0    60   Input ~ 0
+LED[0..5]
+Entry Wire Line
+	9700 4800 9800 4700
+Wire Bus Line
+	9700 4800 6800 4800
+Entry Wire Line
+	9150 4800 9250 4700
+Entry Wire Line
+	8600 4800 8700 4700
+Entry Wire Line
+	8050 4800 8150 4700
+Entry Wire Line
+	7500 4800 7600 4700
+Entry Wire Line
+	6950 4800 7050 4700
+Wire Wire Line
+	7050 4700 7050 3400
+Text Label 7600 4650 1    60   ~ 0
+LED1
+Text Label 8150 4650 1    60   ~ 0
+LED2
+Text Label 8700 4650 1    60   ~ 0
+LED3
+Text Label 9250 4650 1    60   ~ 0
+LED4
+Text Label 9800 4650 1    60   ~ 0
+LED5
+Text Label 2450 2400 3    60   ~ 0
+KEY0
+Text Label 3000 2400 3    60   ~ 0
+KEY1
+Text Label 3550 2400 3    60   ~ 0
+KEY2
+Text Label 4100 2400 3    60   ~ 0
+KEY3
+Text Label 5000 3150 2    60   ~ 0
+KEY4
+Text Label 5000 3750 2    60   ~ 0
+KEY5
+Text Label 5000 4350 2    60   ~ 0
+KEY6
+Text Label 5000 4950 2    60   ~ 0
+KEY7
+Text Label 7050 4650 1    60   ~ 0
+LED0
 $EndSCHEMATC

Commit message: aktuelle Version
Parts:
- D701, D702, D703, D704, D705, D706: footprint (none) -> LEDs:LED_0603
- R701, R702, R704, R706, R708, R710, R712: footprint (none) -> Resistors_SMD:R_0603
- SW701: footprint buttons:Foil_Button -> buttons:TS-015A
- TP734, TP735, TP736, TP737, TP738, TP739, TP740, TP741, TP742, TP743, TP744, TP745, TP746, TP747, TP748: renamed from TP?; footprint (none) -> buttons:TP
Changed lines of the file:
@@
 $EndComp
 $Comp
-L GND #PWR502
+L GND #PWR077
 U 1 1 5807C50C
 P 1500 4800
-F 0 "#PWR502" H 1500 4550 50  0001 C CNN
+F 0 "#PWR077" H 1500 4550 50  0001 C CNN
 F 1 "GND" H 1500 4650 50  0000 C CNN
 F 2 "" H 1500 4800 50  0000 C CNN
@@
 F 0 "SW701" H 1650 4510 50  0000 C CNN
 F 1 "SW_PUSH" H 1500 4320 50  0000 C CNN
-F 2 "buttons:Foil_Button" H 1500 4400 50  0001 C CNN
+F 2 "buttons:TS-015A" H 1500 4400 50  0001 C CNN
 F 3 "" H 1500 4400 50  0000 C CNN
 	1    1500 4400
@@
 Connection ~ 1500 3950
 $Comp
-L +3V3 #PWR501
+L +3V3 #PWR078
 U 1 1 5807C7B5
 P 1500 3350
-F 0 "#PWR501" H 1500 3200 50  0001 C CNN
+F 0 "#PWR078" H 1500 3200 50  0001 C CNN
 F 1 "+3V3" H 1500 3490 50  0000 C CNN
 F 2 "" H 1500 3350 50  0000 C CNN
@@
 F 0 "R701" V 1580 3650 50  0000 C CNN
 F 1 "10k" V 1500 3650 50  0000 C CNN
-F 2 "" V 1430 3650 50  0001 C CNN
+F 2 "Resistors_SMD:R_0603" V 1430 3650 50  0001 C CNN
 F 3 "" H 1500 3650 50  0000 C CNN
 	1    1500 3650
@@
 F 0 "D701" H 7050 3300 50  0000 C CNN
 F 1 "LED" H 7050 3100 50  0000 C CNN
-F 2 "" H 7050 3200 50  0001 C CNN
+F 2 "LEDs:LED_0603" H 7050 3200 50  0001 C CNN
 F 3 "" H 7050 3200 50  0000 C CNN
 	1    7050 3200
@@
 F 0 "D702" H 7600 3300 50  0000 C CNN
 F 1 "LED" H 7600 3100 50  0000 C CNN
-F 2 "" H 7600 3200 50  0001 C CNN
+F 2 "LEDs:LED_0603" H 7600 3200 50  0001 C CNN
 F 3 "" H 7600 3200 50  0000 C CNN
 	1    7600 3200
@@
 F 0 "D703" H 8150 3300 50  0000 C CNN
 F 1 "LED" H 8150 3100 50  0000 C CNN
-F 2 "" H 8150 3200 50  0001 C CNN
+F 2 "LEDs:LED_0603" H 8150 3200 50  0001 C CNN
 F 3 "" H 8150 3200 50  0000 C CNN
 	1    8150 3200
@@
 F 0 "D704" H 8700 3300 50  0000 C CNN
 F 1 "LED" H 8700 3100 50  0000 C CNN
-F 2 "" H 8700 3200 50  0001 C CNN
+F 2 "LEDs:LED_0603" H 8700 3200 50  0001 C CNN
 F 3 "" H 8700 3200 50  0000 C CNN
 	1    8700 3200
@@
 F 0 "D705" H 9250 3300 50  0000 C CNN
 F 1 "LED" H 9250 3100 50  0000 C CNN
-F 2 "" H 9250 3200 50  0001 C CNN
+F 2 "LEDs:LED_0603" H 9250 3200 50  0001 C CNN
 F 3 "" H 9250 3200 50  0000 C CNN
 	1    9250 3200
@@
 F 0 "D706" H 9800 3300 50  0000 C CNN
 F 1 "LED" H 9800 3100 50  0000 C CNN
-F 2 "" H 9800 3200 50  0001 C CNN
+F 2 "LEDs:LED_0603" H 9800 3200 50  0001 C CNN
 F 3 "" H 9800 3200 50  0000 C CNN
 	1    9800 3200
@@
 F 0 "R702" V 7130 2650 50  0000 C CNN
 F 1 "280" V 7050 2650 50  0000 C CNN
-F 2 "" V 6980 2650 50  0001 C CNN
+F 2 "Resistors_SMD:R_0603" V 6980 2650 50  0001 C CNN
 F 3 "" H 7050 2650 50  0000 C CNN
 	1    7050 2650
@@
 F 0 "R704" V 7680 2650 50  0000 C CNN
 F 1 "280" V 7600 2650 50  0000 C CNN
-F 2 "" V 7530 2650 50  0001 C CNN
+F 2 "Resistors_SMD:R_0603" V 7530 2650 50  0001 C CNN
 F 3 "" H 7600 2650 50  0000 C CNN
 	1    7600 2650
@@
 F 0 "R706" V 8230 2650 50  0000 C CNN
 F 1 "280" V 8150 2650 50  0000 C CNN
-F 2 "" V 8080 2650 50  0001 C CNN
+F 2 "Resistors_SMD:R_0603" V 8080 2650 50  0001 C CNN
 F 3 "" H 8150 2650 50  0000 C CNN
 	1    8150 2650
@@
 F 0 "R708" V 8780 2650 50  0000 C CNN
 F 1 "280" V 8700 2650 50  0000 C CNN
-F 2 "" V 8630 2650 50  0001 C CNN
+F 2 "Resistors_SMD:R_0603" V 8630 2650 50  0001 C CNN
 F 3 "" H 8700 2650 50  0000 C CNN
 	1    8700 2650
@@
 F 0 "R710" V 9330 2650 50  0000 C CNN
 F 1 "280" V 9250 2650 50  0000 C CNN
-F 2 "" V 9180 2650 50  0001 C CNN
+F 2 "Resistors_SMD:R_0603" V 9180 2650 50  0001 C CNN
 F 3 "" H 9250 2650 50  0000 C CNN
 	1    9250 2650
@@
 F 0 "R712" V 9880 2650 50  0000 C CNN
 F 1 "280" V 9800 2650 50  0000 C CNN
-F 2 "" V 9730 2650 50  0001 C CNN
+F 2 "Resistors_SMD:R_0603" V 9730 2650 50  0001 C CNN
 F 3 "" H 9800 2650 50  0000 C CNN
 	1    9800 2650
@@
 	9800 2800 9800 3000
 $Comp
-L +3V3 #PWR503
+L +3V3 #PWR079
 U 1 1 580805E8
 P 7050 2300
-F 0 "#PWR503" H 7050 2150 50  0001 C CNN
+F 0 "#PWR079" H 7050 2150 50  0001 C CNN
 F 1 "+3V3" H 7050 2440 50  0000 C CNN
 F 2 "" H 7050 2300 50  0000 C CNN
@@
 	9800 3400 9800 4700
 $Comp
-L TP TP?
+L TP TP743
 U 1 1 585B661A
 P 7050 3775
-F 0 "TP?" H 7050 3815 20  0000 C CNN
+F 0 "TP743" H 7050 3815 20  0000 C CNN
 F 1 "TP" H 7050 3725 60  0001 C CNN
-F 2 "" H 7050 3775 60  0000 C CNN
+F 2 "buttons:TP" H 7050 3775 60  0001 C CNN
 F 3 "" H 7050 3775 60  0000 C CNN
 	1    7050 3775
@@
 $EndComp
 $Comp
-L TP TP?
+L TP TP744
 U 1 1 585B68D9
 P 7600 3775
-F 0 "TP?" H 7600 3815 20  0000 C CNN
+F 0 "TP744" H 7600 3815 20  0000 C CNN
 F 1 "TP" H 7600 3725 60  0001 C CNN
-F 2 "" H 7600 3775 60  0000 C CNN
+F 2 "buttons:TP" H 7600 3775 60  0001 C CNN
 F 3 "" H 7600 3775 60  0000 C CNN
 	1    7600 3775
@@
 $EndComp
 $Comp
-L TP TP?
+L TP TP745
 U 1 1 585B692E
 P 8150 3775
-F 0 "TP?" H 8150 3815 20  0000 C CNN
+F 0 "TP745" H 8150 3815 20  0000 C CNN
 F 1 "TP" H 8150 3725 60  0001 C CNN
-F 2 "" H 8150 3775 60  0000 C CNN
+F 2 "buttons:TP" H 8150 3775 60  0001 C CNN
 F 3 "" H 8150 3775 60  0000 C CNN
 	1    8150 3775
@@
 $EndComp
 $Comp
-L TP TP?
+L TP TP746
 U 1 1 585B6985
 P 8700 3775
-F 0 "TP?" H 8700 3815 20  0000 C CNN
+F 0 "TP746" H 8700 3815 20  0000 C CNN
 F 1 "TP" H 8700 3725 60  0001 C CNN
-F 2 "" H 8700 3775 60  0000 C CNN
+F 2 "buttons:TP" H 8700 3775 60  0001 C CNN
 F 3 "" H 8700 3775 60  0000 C CNN
 	1    8700 3775
@@
 $EndComp
 $Comp
-L TP TP?
+L TP TP747
 U 1 1 585B6D0E
 P 9250 3775
-F 0 "TP?" H 9250 3815 20  0000 C CNN
+F 0 "TP747" H 9250 3815 20  0000 C CNN
 F 1 "TP" H 9250 3725 60  0001 C CNN
-F 2 "" H 9250 3775 60  0000 C CNN
+F 2 "buttons:TP" H 9250 3775 60  0001 C CNN
 F 3 "" H 9250 3775 60  0000 C CNN
 	1    9250 3775
@@
 $EndComp
 $Comp
-L TP TP?
+L TP TP748
 U 1 1 585B6D69
 P 9800 3775
-F 0 "TP?" H 9800 3815 20  0000 C CNN
+F 0 "TP748" H 9800 3815 20  0000 C CNN
 F 1 "TP" H 9800 3725 60  0001 C CNN
-F 2 "" H 9800 3775 60  0000 C CNN
+F 2 "buttons:TP" H 9800 3775 60  0001 C CNN
 F 3 "" H 9800 3775 60  0000 C CNN
 	1    9800 3775
@@
 $EndComp
 $Comp
-L TP TP?
+L TP TP735
 U 1 1 585B7582
 P 2450 2750
-F 0 "TP?" H 2450 2790 20  0000 C CNN
+F 0 "TP735" H 2450 2790 20  0000 C CNN
 F 1 "TP" H 2450 2700 60  0001 C CNN
-F 2 "" H 2450 2750 60  0000 C CNN
+F 2 "buttons:TP" H 2450 2750 60  0001 C CNN
 F 3 "" H 2450 2750 60  0000 C CNN
 	1    2450 2750
@@
 $EndComp
 $Comp
-L TP TP?
+L TP TP736
 U 1 1 585B75E1
 P 3000 2750
-F 0 "TP?" H 3000 2790 20  0000 C CNN
+F 0 "TP736" H 3000 2790 20  0000 C CNN
 F 1 "TP" H 3000 2700 60  0001 C CNN
-F 2 "" H 3000 2750 60  0000 C CNN
+F 2 "buttons:TP" H 3000 2750 60  0001 C CNN
 F 3 "" H 3000 2750 60  0000 C CNN
 	1    3000 2750
@@
 $EndComp
 $Comp
-L TP TP?
+L TP TP737
 U 1 1 585B7642
 P 3550 2750
-F 0 "TP?" H 3550 2790 20  0000 C CNN
+F 0 "TP737" H 3550 2790 20  0000 C CNN
 F 1 "TP" H 3550 2700 60  0001 C CNN
-F 2 "" H 3550 2750 60  0000 C CNN
+F 2 "buttons:TP" H 3550 2750 60  0001 C CNN
 F 3 "" H 3550 2750 60  0000 C CNN
 	1    3550 2750
@@
 $EndComp
 $Comp
-L TP TP?
+L TP TP738
 U 1 1 585B7879
 P 4100 2750
-F 0 "TP?" H 4100 2790 20  0000 C CNN
+F 0 "TP738" H 4100 2790 20  0000 C CNN
 F 1 "TP" H 4100 2700 60  0001 C CNN
-F 2 "" H 4100 2750 60  0000 C CNN
+F 2 "buttons:TP" H 4100 2750 60  0001 C CNN
 F 3 "" H 4100 2750 60  0000 C CNN
 	1    4100 2750
@@
 $EndComp
 $Comp
-L TP TP?
+L TP TP739
 U 1 1 585B78DE
 P 4650 3150
-F 0 "TP?" H 4650 3190 20  0000 C CNN
+F 0 "TP739" H 4650 3190 20  0000 C CNN
 F 1 "TP" H 4650 3100 60  0001 C CNN
-F 2 "" H 4650 3150 60  0000 C CNN
+F 2 "buttons:TP" H 4650 3150 60  0001 C CNN
 F 3 "" H 4650 3150 60  0000 C CNN
 	1    4650 3150
@@
 $EndComp
 $Comp
-L TP TP?
+L TP TP740
 U 1 1 585B7945
 P 4650 3750
-F 0 "TP?" H 4650 3790 20  0000 C CNN
+F 0 "TP740" H 4650 3790 20  0000 C CNN
 F 1 "TP" H 4650 3700 60  0001 C CNN
-F 2 "" H 4650 3750 60  0000 C CNN
+F 2 "buttons:TP" H 4650 3750 60  0001 C CNN
 F 3 "" H 4650 3750 60  0000 C CNN
 	1    4650 3750
@@
 $EndComp
 $Comp
-L TP TP?
+L TP TP741
 U 1 1 585B7C4E
 P 4650 4350
-F 0 "TP?" H 4650 4390 20  0000 C CNN
+F 0 "TP741" H 4650 4390 20  0000 C CNN
 F 1 "TP" H 4650 4300 60  0001 C CNN
-F 2 "" H 4650 4350 60  0000 C CNN
+F 2 "buttons:TP" H 4650 4350 60  0001 C CNN
 F 3 "" H 4650 4350 60  0000 C CNN
 	1    4650 4350
@@
 $EndComp
 $Comp
-L TP TP?
+L TP TP742
 U 1 1 585B7CB9
 P 4650 4950
-F 0 "TP?" H 4650 4990 20  0000 C CNN
+F 0 "TP742" H 4650 4990 20  0000 C CNN
 F 1 "TP" H 4650 4900 60  0001 C CNN
-F 2 "" H 4650 4950 60  0000 C CNN
+F 2 "buttons:TP" H 4650 4950 60  0001 C CNN
 F 3 "" H 4650 4950 60  0000 C CNN
 	1    4650 4950
@@
 $EndComp
 $Comp
-L TP TP?
+L TP TP734
 U 1 1 585B7FE6
 P 1500 3950
-F 0 "TP?" H 1500 3990 20  0000 C CNN
+F 0 "TP734" H 1500 3990 20  0000 C CNN
 F 1 "TP" H 1500 3900 60  0001 C CNN
-F 2 "" H 1500 3950 60  0000 C CNN
+F 2 "buttons:TP" H 1500 3950 60  0001 C CNN
 F 3 "" H 1500 3950 60  0000 C CNN
 	1    1500 3950

Commit message: display placement
The placement of the display connector is set.
Parts:
- D701, D702, D703, D704, D705, D706: symbol LED -> LED-RESCUE-3210retro
Changed lines of the file:
@@
 EESchema Schematic File Version 2
+LIBS:3210retro-rescue
 LIBS:power
 LIBS:device
@@
 Connection ~ 4400 4950
 $Comp
-L LED D701
+L LED-RESCUE-3210retro D701
 U 1 1 5807DD28
 P 7050 3200
+AR Path="/5807DD28" Ref="D701"  Part="1"
+AR Path="/5805F4BA/5807DD28" Ref="D701"  Part="1"
 F 0 "D701" H 7050 3300 50  0000 C CNN
 F 1 "LED" H 7050 3100 50  0000 C CNN
@@
 $EndComp
 $Comp
-L LED D702
+L LED-RESCUE-3210retro D702
 U 1 1 5807DE0F
 P 7600 3200
+AR Path="/5807DE0F" Ref="D702"  Part="1"
+AR Path="/5805F4BA/5807DE0F" Ref="D702"  Part="1"
 F 0 "D702" H 7600 3300 50  0000 C CNN
 F 1 "LED" H 7600 3100 50  0000 C CNN
@@
 $EndComp
 $Comp
-L LED D703
+L LED-RESCUE-3210retro D703
 U 1 1 5807DE69
 P 8150 3200
+AR Path="/5807DE69" Ref="D703"  Part="1"
+AR Path="/5805F4BA/5807DE69" Ref="D703"  Part="1"
 F 0 "D703" H 8150 3300 50  0000 C CNN
 F 1 "LED" H 8150 3100 50  0000 C CNN
@@
 $EndComp
 $Comp
-L LED D704
+L LED-RESCUE-3210retro D704
 U 1 1 5807DEC0
 P 8700 3200
+AR Path="/5807DEC0" Ref="D704"  Part="1"
+AR Path="/5805F4BA/5807DEC0" Ref="D704"  Part="1"
 F 0 "D704" H 8700 3300 50  0000 C CNN
 F 1 "LED" H 8700 3100 50  0000 C CNN
@@
 $EndComp
 $Comp
-L LED D705
+L LED-RESCUE-3210retro D705
 U 1 1 5807DF22
 P 9250 3200
+AR Path="/5807DF22" Ref="D705"  Part="1"
+AR Path="/5805F4BA/5807DF22" Ref="D705"  Part="1"
 F 0 "D705" H 9250 3300 50  0000 C CNN
 F 1 "LED" H 9250 3100 50  0000 C CNN
@@
 $EndComp
 $Comp
-L LED D706
+L LED-RESCUE-3210retro D706
 U 1 1 5807DF8B
 P 9800 3200
+AR Path="/5807DF8B" Ref="D706"  Part="1"
+AR Path="/5805F4BA/5807DF8B" Ref="D706"  Part="1"
 F 0 "D706" H 9800 3300 50  0000 C CNN
 F 1 "LED" H 9800 3100 50  0000 C CNN
