File: INPUT.sch (KiCad schematic (older format))
At the start: 41 parts, among them SW701 SW_PUSH, SW702 C, SW703 1, SW704 4ghi, SW705 7pqrs, SW706 -, SW707 2abc, SW708 5jkl, SW709 8tuv, SW710 UP, SW711 3def, SW712 6mno, SW713 9wxyz, SW714 *+, SW715 DOWN, SW716 0space, SW717 #up

Commit message: Prepare for two battery types NiMH battery for using the original battery pack LiPo battery for using long lasting modern battery
Parts:
- gave numbers to parts that had none: 2
Changed lines of the file:
@@
 EESchema Schematic File Version 2
-LIBS:3210retro-rescue
-LIBS:power
-LIBS:device
-LIBS:transistors
-LIBS:conn
-LIBS:linear
-LIBS:regul
-LIBS:74xx
-LIBS:cmos4000
-LIBS:adc-dac
-LIBS:memory
-LIBS:xilinx
-LIBS:microcontrollers
-LIBS:dsp
-LIBS:microchip
-LIBS:analog_switches
-LIBS:motorola
-LIBS:texas
-LIBS:intel
-LIBS:audio
-LIBS:interface
-LIBS:digital-audio
-LIBS:philips
-LIBS:display
-LIBS:cypress
-LIBS:siliconi
-LIBS:opto
-LIBS:atmel
-LIBS:contrib
-LIBS:valves
 LIBS:a7
 LIBS:ft232rl
@@
 LIBS:sn74avc2t244
 LIBS:lsm9ds1
+LIBS:WM8960CGEFL
+LIBS:tps61021a
+LIBS:bq24400
+LIBS:power
+LIBS:device
+LIBS:transistors
+LIBS:conn
+LIBS:linear
+LIBS:regul
+LIBS:74xx
+LIBS:cmos4000
+LIBS:adc-dac
+LIBS:memory
+LIBS:xilinx
+LIBS:microcontrollers
+LIBS:dsp
+LIBS:microchip
+LIBS:analog_switches
+LIBS:motorola
+LIBS:texas
+LIBS:intel
+LIBS:audio
+LIBS:interface
+LIBS:digital-audio
+LIBS:philips
+LIBS:display
+LIBS:cypress
+LIBS:siliconi
+LIBS:opto
+LIBS:atmel
+LIBS:contrib
+LIBS:valves
 LIBS:3210retro-cache
 EELAYER 25 0
@@
 $EndComp
 $Comp
-L GND #PWR089
+L GND #PWR702
 U 1 1 5807C50C
 P 1700 4800
-F 0 "#PWR089" H 1700 4550 50  0001 C CNN
+F 0 "#PWR702" H 1700 4550 50  0001 C CNN
 F 1 "GND" H 1700 4650 50  0000 C CNN
 F 2 "" H 1700 4800 50  0000 C CNN
@@
 Connection ~ 1700 3950
 $Comp
-L +3V3 #PWR090
+L +3V3 #PWR701
 U 1 1 5807C7B5
 P 1700 3350
-F 0 "#PWR090" H 1700 3200 50  0001 C CNN
+F 0 "#PWR701" H 1700 3200 50  0001 C CNN
 F 1 "+3V3" H 1700 3490 50  0000 C CNN
 F 2 "" H 1700 3350 50  0000 C CNN
@@
 	9800 2800 9800 3000
 $Comp
-L +3V3 #PWR091
+L +3V3 #PWR703
 U 1 1 580805E8
 P 7050 2300
-F 0 "#PWR091" H 7050 2150 50  0001 C CNN
+F 0 "#PWR703" H 7050 2150 50  0001 C CNN
 F 1 "+3V3" H 7050 2440 50  0000 C CNN
 F 2 "" H 7050 2300 50  0000 C CNN
@@
 Connection ~ 9250 4050
 $Comp
-L MMBF170 Q?
+L MMBF170 Q701
 U 1 1 5942422F
 P 9700 4450
-F 0 "Q?" H 9900 4525 50  0000 L CNN
+F 0 "Q701" H 9900 4525 50  0000 L CNN
 F 1 "MMBF170" H 9900 4450 50  0000 L CNN
 F 2 "SOT-23" H 9900 4375 50  0000 L CIN
@@
 $EndComp
 $Comp
-L R R?
+L R R711
 U 1 1 594243DC
 P 9300 4500
-F 0 "R?" V 9380 4500 50  0000 C CNN
+F 0 "R711" V 9380 4500 50  0000 C CNN
 F 1 "280" V 9300 4500 50  0000 C CNN
 F 2 "Resistors_SMD:R_0603" V 9230 4500 50  0001 C CNN
@@
 	9150 4500 9100 4500
 $Comp
-L GND #PWR?
+L GND #PWR704
 U 1 1 5942469E
 P 9800 4700
-F 0 "#PWR?" H 9800 4450 50  0001 C CNN
+F 0 "#PWR704" H 9800 4450 50  0001 C CNN
 F 1 "GND" H 9800 4550 50  0000 C CNN
 F 2 "" H 9800 4700 50  0000 C CNN

Commit message: Changed several voltage rail connections Removed non existing rails Added circuit for NiMH charging
Parts:
- removed D701, D702, D703, D704, D705, D706: LED, LEDs:LED_0603, symbol LED-RESCUE-3210retro
- added D701, D702, D703, D704, D705, D706: LED, symbol LED
- renumbered R704 to R703, R706 to R704, R708 to R705, R710 to R706, R711 to R707, R712 to R708, TP734 to TP701, TP735 to TP702, TP736 to TP703, TP737 to TP704, TP738 to TP705, TP739 to TP706, TP740 to TP707, TP741 to TP708, TP742 to TP709
Connections:
- net labels added: NVCC_3V3, VSNVS
- net labels removed: +3V3
Changed lines of the file:
@@
 $EndComp
 $Comp
-L GND #PWR702
+L GND #PWR0129
 U 1 1 5807C50C
 P 1700 4800
-F 0 "#PWR702" H 1700 4550 50  0001 C CNN
+F 0 "#PWR0129" H 1700 4550 50  0001 C CNN
 F 1 "GND" H 1700 4650 50  0000 C CNN
 F 2 "" H 1700 4800 50  0000 C CNN
@@
 Connection ~ 1700 3950
 $Comp
-L +3V3 #PWR701
-U 1 1 5807C7B5
-P 1700 3350
-F 0 "#PWR701" H 1700 3200 50  0001 C CNN
-F 1 "+3V3" H 1700 3490 50  0000 C CNN
-F 2 "" H 1700 3350 50  0000 C CNN
-F 3 "" H 1700 3350 50  0000 C CNN
-	1    1700 3350
-	1    0    0    -1
-$EndComp
-$Comp
 L R R701
 U 1 1 5807C9B7
@@
 Connection ~ 4600 4950
 $Comp
-L LED-RESCUE-3210retro D701
-U 1 1 5807DD28
-P 7050 3200
-AR Path="/5807DD28" Ref="D701"  Part="1"
-AR Path="/5805F4BA/5807DD28" Ref="D701"  Part="1"
-F 0 "D701" H 7050 3300 50  0000 C CNN
-F 1 "LED" H 7050 3100 50  0000 C CNN
-F 2 "LEDs:LED_0603" H 7050 3200 50  0001 C CNN
-F 3 "" H 7050 3200 50  0000 C CNN
-	1    7050 3200
-	0    -1   -1   0
-$EndComp
-$Comp
-L LED-RESCUE-3210retro D702
-U 1 1 5807DE0F
-P 7600 3200
-AR Path="/5807DE0F" Ref="D702"  Part="1"
-AR Path="/5805F4BA/5807DE0F" Ref="D702"  Part="1"
-F 0 "D702" H 7600 3300 50  0000 C CNN
-F 1 "LED" H 7600 3100 50  0000 C CNN
-F 2 "LEDs:LED_0603" H 7600 3200 50  0001 C CNN
-F 3 "" H 7600 3200 50  0000 C CNN
-	1    7600 3200
-	0    -1   -1   0
-$EndComp
-$Comp
-L LED-RESCUE-3210retro D703
-U 1 1 5807DE69
-P 8150 3200
-AR Path="/5807DE69" Ref="D703"  Part="1"
-AR Path="/5805F4BA/5807DE69" Ref="D703"  Part="1"
-F 0 "D703" H 8150 3300 50  0000 C CNN
-F 1 "LED" H 8150 3100 50  0000 C CNN
-F 2 "LEDs:LED_0603" H 8150 3200 50  0001 C CNN
-F 3 "" H 8150 3200 50  0000 C CNN
-	1    8150 3200
-	0    -1   -1   0
-$EndComp
-$Comp
-L LED-RESCUE-3210retro D704
-U 1 1 5807DEC0
-P 8700 3200
-AR Path="/5807DEC0" Ref="D704"  Part="1"
-AR Path="/5805F4BA/5807DEC0" Ref="D704"  Part="1"
-F 0 "D704" H 8700 3300 50  0000 C CNN
-F 1 "LED" H 8700 3100 50  0000 C CNN
-F 2 "LEDs:LED_0603" H 8700 3200 50  0001 C CNN
-F 3 "" H 8700 3200 50  0000 C CNN
-	1    8700 3200
-	0    -1   -1   0
-$EndComp
-$Comp
-L LED-RESCUE-3210retro D705
-U 1 1 5807DF22
-P 9250 3200
-AR Path="/5807DF22" Ref="D705"  Part="1"
-AR Path="/5805F4BA/5807DF22" Ref="D705"  Part="1"
-F 0 "D705" H 9250 3300 50  0000 C CNN
-F 1 "LED" H 9250 3100 50  0000 C CNN
-F 2 "LEDs:LED_0603" H 9250 3200 50  0001 C CNN
-F 3 "" H 9250 3200 50  0000 C CNN
-	1    9250 3200
-	0    -1   -1   0
-$EndComp
-$Comp
-L LED-RESCUE-3210retro D706
-U 1 1 5807DF8B
-P 9800 3200
-AR Path="/5807DF8B" Ref="D706"  Part="1"
-AR Path="/5805F4BA/5807DF8B" Ref="D706"  Part="1"
-F 0 "D706" H 9800 3300 50  0000 C CNN
-F 1 "LED" H 9800 3100 50  0000 C CNN
-F 2 "LEDs:LED_0603" H 9800 3200 50  0001 C CNN
-F 3 "" H 9800 3200 50  0000 C CNN
-	1    9800 3200
-	0    -1   -1   0
-$EndComp
-$Comp
 L R R702
 U 1 1 5807E47A
@@
 	7050 2800 7050 3000
 $Comp
-L R R704
+L R R703
 U 1 1 5807E634
 P 7600 2650
-F 0 "R704" V 7680 2650 50  0000 C CNN
+F 0 "R703" V 7680 2650 50  0000 C CNN
 F 1 "280" V 7600 2650 50  0000 C CNN
 F 2 "Resistors_SMD:R_0603" V 7530 2650 50  0001 C CNN
@@
 $EndComp
 $Comp
-L R R706
+L R R704
 U 1 1 5807E6A0
 P 8150 2650
-F 0 "R706" V 8230 2650 50  0000 C CNN
+F 0 "R704" V 8230 2650 50  0000 C CNN
 F 1 "280" V 8150 2650 50  0000 C CNN
 F 2 "Resistors_SMD:R_0603" V 8080 2650 50  0001 C CNN
@@
 $EndComp
 $Comp
-L R R708
+L R R705
 U 1 1 5807E785
 P 8700 2650
-F 0 "R708" V 8780 2650 50  0000 C CNN
+F 0 "R705" V 8780 2650 50  0000 C CNN
 F 1 "280" V 8700 2650 50  0000 C CNN
 F 2 "Resistors_SMD:R_0603" V 8630 2650 50  0001 C CNN
@@
 $EndComp
 $Comp
-L R R710
+L R R706
 U 1 1 5807E78B
 P 9250 2650
-F 0 "R710" V 9330 2650 50  0000 C CNN
+F 0 "R706" V 9330 2650 50  0000 C CNN
 F 1 "280" V 9250 2650 50  0000 C CNN
 F 2 "Resistors_SMD:R_0603" V 9180 2650 50  0001 C CNN
@@
 $EndComp
 $Comp
-L R R712
+L R R708
 U 1 1 5807E791
 P 9800 2650
-F 0 "R712" V 9880 2650 50  0000 C CNN
+F 0 "R708" V 9880 2650 50  0000 C CNN
 F 1 "280" V 9800 2650 50  0000 C CNN
 F 2 "Resistors_SMD:R_0603" V 9730 2650 50  0001 C CNN
@@
 Wire Wire Line
 	9800 2800 9800 3000
-$Comp
-L +3V3 #PWR703
-U 1 1 580805E8
-P 7050 2300
-F 0 "#PWR703" H 7050 2150 50  0001 C CNN
-F 1 "+3V3" H 7050 2440 50  0000 C CNN
-F 2 "" H 7050 2300 50  0000 C CNN
-F 3 "" H 7050 2300 50  0000 C CNN
-	1    7050 2300
-	1    0    0    -1
-$EndComp
 Wire Wire Line
 	7050 2300 7050 2500
@@
 Connection ~ 9250 2400
 $Comp
-L TP TP735
+L TP TP702
 U 1 1 585B7582
 P 2650 2750
-F 0 "TP735" H 2650 2790 20  0000 C CNN
+F 0 "TP702" H 2650 2790 20  0000 C CNN
 F 1 "TP" H 2650 2700 60  0001 C CNN
 F 2 "buttons:TP" H 2650 2750 60  0001 C CNN
@@
 $EndComp
 $Comp
-L TP TP736
+L TP TP703
 U 1 1 585B75E1
 P 3200 2750
-F 0 "TP736" H 3200 2790 20  0000 C CNN
+F 0 "TP703" H 3200 2790 20  0000 C CNN
 F 1 "TP" H 3200 2700 60  0001 C CNN
 F 2 "buttons:TP" H 3200 2750 60  0001 C CNN
@@
 $EndComp
 $Comp
-L TP TP737
+L TP TP704
 U 1 1 585B7642
 P 3750 2750
-F 0 "TP737" H 3750 2790 20  0000 C CNN
+F 0 "TP704" H 3750 2790 20  0000 C CNN
 F 1 "TP" H 3750 2700 60  0001 C CNN
 F 2 "buttons:TP" H 3750 2750 60  0001 C CNN
@@
 $EndComp
 $Comp
-L TP TP738
+L TP TP705
 U 1 1 585B7879
 P 4300 2750
-F 0 "TP738" H 4300 2790 20  0000 C CNN
+F 0 "TP705" H 4300 2790 20  0000 C CNN
 F 1 "TP" H 4300 2700 60  0001 C CNN
 F 2 "buttons:TP" H 4300 2750 60  0001 C CNN
@@
 $EndComp
 $Comp
-L TP TP739
+L TP TP706
 U 1 1 585B78DE
 P 4850 3150
-F 0 "TP739" H 4850 3190 20  0000 C CNN
+F 0 "TP706" H 4850 3190 20  0000 C CNN
 F 1 "TP" H 4850 3100 60  0001 C CNN
 F 2 "buttons:TP" H 4850 3150 60  0001 C CNN
@@
 $EndComp
 $Comp
-L TP TP740
+L TP TP707
 U 1 1 585B7945
 P 4850 3750
-F 0 "TP740" H 4850 3790 20  0000 C CNN
+F 0 "TP707" H 4850 3790 20  0000 C CNN
 F 1 "TP" H 4850 3700 60  0001 C CNN
 F 2 "buttons:TP" H 4850 3750 60  0001 C CNN
@@
 $EndComp
 $Comp
-L TP TP741
+L TP TP708
 U 1 1 585B7C4E
 P 4850 4350
-F 0 "TP741" H 4850 4390 20  0000 C CNN
+F 0 "TP708" H 4850 4390 20  0000 C CNN
 F 1 "TP" H 4850 4300 60  0001 C CNN
 F 2 "buttons:TP" H 4850 4350 60  0001 C CNN
@@
 $EndComp
 $Comp
-L TP TP742
+L TP TP709
 U 1 1 585B7CB9
 P 4850 4950
-F 0 "TP742" H 4850 4990 20  0000 C CNN
+F 0 "TP709" H 4850 4990 20  0000 C CNN
 F 1 "TP" H 4850 4900 60  0001 C CNN
 F 2 "buttons:TP" H 4850 4950 60  0001 C CNN
@@
 $EndComp
 $Comp
-L TP TP734
+L TP TP701
 U 1 1 585B7FE6
 P 1700 3950
-F 0 "TP734" H 1700 3990 20  0000 C CNN
+F 0 "TP701" H 1700 3990 20  0000 C CNN
 F 1 "TP" H 1700 3900 60  0001 C CNN
 F 2 "buttons:TP" H 1700 3950 60  0001 C CNN
@@
 $EndComp
 $Comp
-L R R711
+L R R707
 U 1 1 594243DC
 P 9300 4500
-F 0 "R711" V 9380 4500 50  0000 C CNN
+F 0 "R707" V 9380 4500 50  0000 C CNN
 F 1 "280" V 9300 4500 50  0000 C CNN
 F 2 "Resistors_SMD:R_0603" V 9230 4500 50  0001 C CNN
@@
 	9150 4500 9100 4500
 $Comp
-L GND #PWR704
+L GND #PWR0130
 U 1 1 5942469E
 P 9800 4700
-F 0 "#PWR704" H 9800 4450 50  0001 C CNN
+F 0 "#PWR0130" H 9800 4450 50  0001 C CNN
 F 1 "GND" H 9800 4550 50  0000 C CNN
 F 2 "" H 9800 4700 50  0000 C CNN
@@
 	9800 4700 9800 4650
 Connection ~ 9800 4050
+$Comp
+L NVCC_3V3 #PWR0131
+U 1 1 5962C5D6
+P 7050 2300
+F 0 "#PWR0131" H 7050 2150 50  0001 C CNN
+F 1 "NVCC_3V3" H 7050 2450 50  0000 C CNN
+F 2 "" H 7050 2300 50  0001 C CNN
+F 3 "" H 7050 2300 50  0001 C CNN
+	1    7050 2300
+	1    0    0    -1
+$EndComp
+$Comp
+L LED D701
+U 1 1 5962C7F0
+P 7050 3200
+F 0 "D701" H 7050 3300 50  0000 C CNN
+F 1 "LED" H 7050 3100 50  0000 C CNN
+F 2 "" H 7050 3200 50  0000 C CNN
+F 3 "" H 7050 3200 50  0000 C CNN
+	1    7050 3200
+	0    -1   -1   0
+$EndComp
+$Comp
+L LED D702
+U 1 1 5962C95B
+P 7600 3200
+F 0 "D702" H 7600 3300 50  0000 C CNN
+F 1 "LED" H 7600 3100 50  0000 C CNN
+F 2 "" H 7600 3200 50  0000 C CNN
+F 3 "" H 7600 3200 50  0000 C CNN
+	1    7600 3200
+	0    -1   -1   0
+$EndComp
+$Comp
+L LED D703
+U 1 1 5962C9E4
+P 8150 3200
+F 0 "D703" H 8150 3300 50  0000 C CNN
+F 1 "LED" H 8150 3100 50  0000 C CNN
+F 2 "" H 8150 3200 50  0000 C CNN
+F 3 "" H 8150 3200 50  0000 C CNN
+	1    8150 3200
+	0    -1   -1   0
+$EndComp
+$Comp
+L LED D704
+U 1 1 5962CA9C
+P 8700 3200
+F 0 "D704" H 8700 3300 50  0000 C CNN
+F 1 "LED" H 8700 3100 50  0000 C CNN
+F 2 "" H 8700 3200 50  0000 C CNN
+F 3 "" H 8700 3200 50  0000 C CNN
+	1    8700 3200
+	0    -1   -1   0
+$EndComp
+$Comp
+L LED D705
+U 1 1 5962CB2D
+P 9250 3200
+F 0 "D705" H 9250 3300 50  0000 C CNN
+F 1 "LED" H 9250 3100 50  0000 C CNN
+F 2 "" H 9250 3200 50  0000 C CNN
+F 3 "" H 9250 3200 50  0000 C CNN
+	1    9250 3200
+	0    -1   -1   0
+$EndComp
+$Comp
+L LED D706
+U 1 1 5962CBED
+P 9800 3200
+F 0 "D706" H 9800 3300 50  0000 C CNN
+F 1 "LED" H 9800 3100 50  0000 C CNN
+F 2 "" H 9800 3200 50  0000 C CNN
+F 3 "" H 9800 3200 50  0000 C CNN
+	1    9800 3200
+	0    -1   -1   0
+$EndComp
+$Comp
+L VSNVS #PWR0132
+U 1 1 5962CD0E
+P 1700 3350
+F 0 "#PWR0132" H 1700 3200 50  0001 C CNN
+F 1 "VSNVS" H 1700 3500 50  0000 C CNN
+F 2 "" H 1700 3350 50  0001 C CNN
+F 3 "" H 1700 3350 50  0001 C CNN
+	1    1700 3350
+	1    0    0    -1
+$EndComp
 $EndSCHEMATC
