File: INPUT.sch (KiCad schematic (older format))
At the start: 41 parts, among them Q701 MMBF170, SW701 SW_PUSH, SW702 C, SW703 1, SW704 4ghi, SW705 7pqrs, SW706 -, SW707 2abc, SW708 5jkl, SW709 8tuv, SW710 UP, SW711 3def, SW712 6mno, SW713 9wxyz, SW714 *+, SW715 DOWN, SW716 0space, SW717 #up

Commit message: This branch moves from i.mx7 to STM32F4 CPU to be finished for Hackaday Prize 2017
Parts:
- D701, D702, D703, D704, D705, D706: symbol LED -> LED-RESCUE-3210retro
- Q701: symbol MMBF170 -> MMBF170-RESCUE-3210retro
Changed lines of the file:
@@
 EESchema Schematic File Version 2
+LIBS:3210retro-rescue
 LIBS:a7
 LIBS:ft232rl
@@
 LIBS:contrib
 LIBS:valves
+LIBS:stm32
 LIBS:3210retro-cache
-EELAYER 25 0
+EELAYER 26 0
 EELAYER END
 $Descr A3 16535 11693
 encoding utf-8
-Sheet 7 13
+Sheet 7 10
 Title "Nokia 3210 Retrofit"
 Date "2017-06-15"
@@
 Connection ~ 9250 4050
 $Comp
-L MMBF170 Q701
+L MMBF170-RESCUE-3210retro Q701
 U 1 1 5942422F
 P 9700 4450
@@
 $EndComp
 $Comp
-L LED D701
+L LED-RESCUE-3210retro D701
 U 1 1 5962C7F0
 P 7050 3200
@@
 $EndComp
 $Comp
-L LED D702
+L LED-RESCUE-3210retro D702
 U 1 1 5962C95B
 P 7600 3200
@@
 $EndComp
 $Comp
-L LED D703
+L LED-RESCUE-3210retro D703
 U 1 1 5962C9E4
 P 8150 3200
@@
 $EndComp
 $Comp
-L LED D704
+L LED-RESCUE-3210retro D704
 U 1 1 5962CA9C
 P 8700 3200
@@
 $EndComp
 $Comp
-L LED D705
+L LED-RESCUE-3210retro D705
 U 1 1 5962CB2D
 P 9250 3200
@@
 $EndComp
 $Comp
-L LED D706
+L LED-RESCUE-3210retro D706
 U 1 1 5962CBED
 P 9800 3200

Commit message: Modification for STM32 adaption
For the Hackaday Prize 2017 I decided to switch to STM32 as CPU

*Power system was modified to just contain the charge IC,
*Boost converter for high voltage peripherals
*Buck converter for 3V3 for CPU and switchable NVCC_3V3
   for peripherie

CPU signals are routed and pinmux is done in firmware folder.

SD-Card has 4bit Interface

WiFi module ESP8266 is connected via UART

Wolfson Ausio codec is connected via SAI

Two digital microphones for noise canceling

Rumble Motor driver

LCD is connected via it's own I2C interface
Parts:
- R701, R702, R703, R704, R705, R706, R707, R708: footprint Resistors_SMD:R_0402 -> Resistors_SMD:R_0402_NoSilk
- SW701: footprint NokiaRetroFit:TS-015A -> Resistors_SMD:R_0402_NoSilk
Changed lines of the file:
@@
 EESchema Schematic File Version 2
-LIBS:3210retro-rescue
 LIBS:a7
 LIBS:ft232rl
@@
 LIBS:contrib
 LIBS:valves
-LIBS:stm32
+LIBS:tps62742
+LIBS:WM8994ECS
 LIBS:3210retro-cache
 EELAYER 26 0
 EELAYER END
-$Descr A3 16535 11693
+$Descr A4 11693 8268
 encoding utf-8
 Sheet 7 10
 Title "Nokia 3210 Retrofit"
-Date "2017-06-15"
-Rev "2"
+Date "2017-09-07"
+Rev "3"
 Comp "www.kurzschluss-blog.de"
-Comment1 "Retrofitting board for Nokia 3210 mobile phone"
-Comment2 ""
+Comment1 "Retro fitting board for Nokia 3210 mobile phone"
+Comment2 "STM32 Version"
 Comment3 ""
 Comment4 ""
@@
 F 0 "SW701" H 1850 4510 50  0000 C CNN
 F 1 "SW_PUSH" H 1700 4320 50  0000 C CNN
-F 2 "NokiaRetroFit:TS-015A" H 1700 4400 50  0001 C CNN
+F 2 "Resistors_SMD:R_0402_NoSilk" H 1700 4400 50  0001 C CNN
 F 3 "" H 1700 4400 50  0000 C CNN
 	1    1700 4400
@@
 F 0 "R701" V 1780 3650 50  0000 C CNN
 F 1 "10k" V 1700 3650 50  0000 C CNN
-F 2 "Resistors_SMD:R_0402" V 1630 3650 50  0001 C CNN
+F 2 "Resistors_SMD:R_0402_NoSilk" V 1630 3650 50  0001 C CNN
 F 3 "" H 1700 3650 50  0000 C CNN
 	1    1700 3650
@@
 F 0 "R702" V 7130 2650 50  0000 C CNN
 F 1 "280" V 7050 2650 50  0000 C CNN
-F 2 "Resistors_SMD:R_0402" V 6980 2650 50  0001 C CNN
+F 2 "Resistors_SMD:R_0402_NoSilk" V 6980 2650 50  0001 C CNN
 F 3 "" H 7050 2650 50  0000 C CNN
 	1    7050 2650
@@
 F 0 "R703" V 7680 2650 50  0000 C CNN
 F 1 "280" V 7600 2650 50  0000 C CNN
-F 2 "Resistors_SMD:R_0402" V 7530 2650 50  0001 C CNN
+F 2 "Resistors_SMD:R_0402_NoSilk" V 7530 2650 50  0001 C CNN
 F 3 "" H 7600 2650 50  0000 C CNN
 	1    7600 2650
@@
 F 0 "R704" V 8230 2650 50  0000 C CNN
 F 1 "280" V 8150 2650 50  0000 C CNN
-F 2 "Resistors_SMD:R_0402" V 8080 2650 50  0001 C CNN
+F 2 "Resistors_SMD:R_0402_NoSilk" V 8080 2650 50  0001 C CNN
 F 3 "" H 8150 2650 50  0000 C CNN
 	1    8150 2650
@@
 F 0 "R705" V 8780 2650 50  0000 C CNN
 F 1 "280" V 8700 2650 50  0000 C CNN
-F 2 "Resistors_SMD:R_0402" V 8630 2650 50  0001 C CNN
+F 2 "Resistors_SMD:R_0402_NoSilk" V 8630 2650 50  0001 C CNN
 F 3 "" H 8700 2650 50  0000 C CNN
 	1    8700 2650
@@
 F 0 "R706" V 9330 2650 50  0000 C CNN
 F 1 "280" V 9250 2650 50  0000 C CNN
-F 2 "Resistors_SMD:R_0402" V 9180 2650 50  0001 C CNN
+F 2 "Resistors_SMD:R_0402_NoSilk" V 9180 2650 50  0001 C CNN
 F 3 "" H 9250 2650 50  0000 C CNN
 	1    9250 2650
@@
 F 0 "R708" V 9880 2650 50  0000 C CNN
 F 1 "280" V 9800 2650 50  0000 C CNN
-F 2 "Resistors_SMD:R_0402" V 9730 2650 50  0001 C CNN
+F 2 "Resistors_SMD:R_0402_NoSilk" V 9730 2650 50  0001 C CNN
 F 3 "" H 9800 2650 50  0000 C CNN
 	1    9800 2650
@@
 F 0 "R707" V 9380 4500 50  0000 C CNN
 F 1 "280" V 9300 4500 50  0000 C CNN
-F 2 "Resistors_SMD:R_0402" V 9230 4500 50  0001 C CNN
+F 2 "Resistors_SMD:R_0402_NoSilk" V 9230 4500 50  0001 C CNN
 F 3 "" H 9300 4500 50  0000 C CNN
 	1    9300 4500

Commit message: Placed a lot of components and routed the audio codec
The BGA of tha audio chipset is to small for regualr technology.
We do not use all of the pins of the chip so we ignore the other
pads and escape throug the balls of the other pad.
Parts:
- SW701: footprint Resistors_SMD:R_0402_NoSilk -> NokiaRetroFit:TS-015A
Changed lines of the file:
@@
 LIBS:contrib
 LIBS:valves
-LIBS:tps62742
-LIBS:WM8994ECS
+LIBS:stm32
 LIBS:3210retro-cache
 EELAYER 26 0
@@
 F 0 "SW701" H 1850 4510 50  0000 C CNN
 F 1 "SW_PUSH" H 1700 4320 50  0000 C CNN
-F 2 "Resistors_SMD:R_0402_NoSilk" H 1700 4400 50  0001 C CNN
+F 2 "NokiaRetroFit:TS-015A" H 1700 4400 50  0001 C CNN
 F 3 "" H 1700 4400 50  0000 C CNN
 	1    1700 4400

Commit message: Revision 1 of Layout
6layer board
through-hole via only (0.5/0.3mm drill)
0.2mm track width

https://hackaday.io/project/21263-nokia-3210-retro-fit-board/log/66914-prototype-pcb-done-there-comes-the-review
Parts:
- removed TP701, TP702, TP703, TP704, TP705, TP706, TP707, TP708, TP709: TP, NokiaRetroFit:TP, symbol TP
Connections:
- net labels added: 3V3
- net labels removed: VSNVS
Changed lines of the file:
@@
 	2900 4900 2950 4950
-Wire Wire Line
-	2950 4950 5550 4950
 Wire Wire Line
 	3500 4950 3450 4900
@@
 	9800 2400 9800 2500
 Connection ~ 9250 2400
-$Comp
-L TP TP702
-U 1 1 585B7582
-P 2650 2750
-F 0 "TP702" H 2650 2790 20  0000 C CNN
-F 1 "TP" H 2650 2700 60  0001 C CNN
-F 2 "NokiaRetroFit:TP" H 2650 2750 60  0001 C CNN
-F 3 "" H 2650 2750 60  0000 C CNN
-	1    2650 2750
-	1    0    0    -1
-$EndComp
-$Comp
-L TP TP703
-U 1 1 585B75E1
-P 3200 2750
-F 0 "TP703" H 3200 2790 20  0000 C CNN
-F 1 "TP" H 3200 2700 60  0001 C CNN
-F 2 "NokiaRetroFit:TP" H 3200 2750 60  0001 C CNN
-F 3 "" H 3200 2750 60  0000 C CNN
-	1    3200 2750
-	1    0    0    -1
-$EndComp
-$Comp
-L TP TP704
-U 1 1 585B7642
-P 3750 2750
-F 0 "TP704" H 3750 2790 20  0000 C CNN
-F 1 "TP" H 3750 2700 60  0001 C CNN
-F 2 "NokiaRetroFit:TP" H 3750 2750 60  0001 C CNN
-F 3 "" H 3750 2750 60  0000 C CNN
-	1    3750 2750
-	1    0    0    -1
-$EndComp
-$Comp
-L TP TP705
-U 1 1 585B7879
-P 4300 2750
-F 0 "TP705" H 4300 2790 20  0000 C CNN
-F 1 "TP" H 4300 2700 60  0001 C CNN
-F 2 "NokiaRetroFit:TP" H 4300 2750 60  0001 C CNN
-F 3 "" H 4300 2750 60  0000 C CNN
-	1    4300 2750
-	1    0    0    -1
-$EndComp
-$Comp
-L TP TP706
-U 1 1 585B78DE
-P 4850 3150
-F 0 "TP706" H 4850 3190 20  0000 C CNN
-F 1 "TP" H 4850 3100 60  0001 C CNN
-F 2 "NokiaRetroFit:TP" H 4850 3150 60  0001 C CNN
-F 3 "" H 4850 3150 60  0000 C CNN
-	1    4850 3150
-	1    0    0    -1
-$EndComp
-$Comp
-L TP TP707
-U 1 1 585B7945
-P 4850 3750
-F 0 "TP707" H 4850 3790 20  0000 C CNN
-F 1 "TP" H 4850 3700 60  0001 C CNN
-F 2 "NokiaRetroFit:TP" H 4850 3750 60  0001 C CNN
-F 3 "" H 4850 3750 60  0000 C CNN
-	1    4850 3750
-	1    0    0    -1
-$EndComp
-$Comp
-L TP TP708
-U 1 1 585B7C4E
-P 4850 4350
-F 0 "TP708" H 4850 4390 20  0000 C CNN
-F 1 "TP" H 4850 4300 60  0001 C CNN
-F 2 "NokiaRetroFit:TP" H 4850 4350 60  0001 C CNN
-F 3 "" H 4850 4350 60  0000 C CNN
-	1    4850 4350
-	1    0    0    -1
-$EndComp
-$Comp
-L TP TP709
-U 1 1 585B7CB9
-P 4850 4950
-F 0 "TP709" H 4850 4990 20  0000 C CNN
-F 1 "TP" H 4850 4900 60  0001 C CNN
-F 2 "NokiaRetroFit:TP" H 4850 4950 60  0001 C CNN
-F 3 "" H 4850 4950 60  0000 C CNN
-	1    4850 4950
-	1    0    0    -1
-$EndComp
-$Comp
-L TP TP701
-U 1 1 585B7FE6
-P 1700 3950
-F 0 "TP701" H 1700 3990 20  0000 C CNN
-F 1 "TP" H 1700 3900 60  0001 C CNN
-F 2 "NokiaRetroFit:TP" H 1700 3950 60  0001 C CNN
-F 3 "" H 1700 3950 60  0000 C CNN
-	1    1700 3950
-	1    0    0    -1
-$EndComp
 Entry Wire Line
 	2550 1800 2650 1900
@@
 	0    -1   -1   0
 $EndComp
-$Comp
-L VSNVS #PWR0132
-U 1 1 5962CD0E
+Wire Wire Line
+	2950 4950 5550 4950
+$Comp
+L 3V3 #PWR03
+U 1 1 59B553CA
 P 1700 3350
-F 0 "#PWR0132" H 1700 3200 50  0001 C CNN
-F 1 "VSNVS" H 1700 3500 50  0000 C CNN
+F 0 "#PWR03" H 1700 3200 50  0001 C CNN
+F 1 "3V3" H 1717 3523 50  0000 C CNN
 F 2 "" H 1700 3350 50  0001 C CNN
 F 3 "" H 1700 3350 50  0001 C CNN
