File: MEMORY.sch (KiCad schematic (older format))
At the start: 31 parts, among them J901 MICRO_SD, U201 STM32F439NIH6, U301 IS42S16400J

Commit message: aktuelle Version
Parts:
- added RP901, RP902, RP903, RP904, RP905: 100, Resistors_SMD:R_Array_Convex_8x0602, symbol R_PACK8
- C301, C302, C303, C304, C305, C306, C307, C903, C904: footprint (none) -> Capacitors_SMD:C_0603
- R910, R911, R912, R913, R914, R915, R916: footprint (none) -> Resistors_SMD:R_0603
- TP901, TP902, TP903, TP904, TP905, TP906, TP907, TP908, TP909, TP910, TP911, TP912: renamed from TP?; footprint (none) -> buttons:TP
Connections:
- net at U201.A5 (PE1/FMC_NBL1): now also RP905.8 (P8); no longer U301.15 (LDQM)
- net at U201.A6 (PE0/FMC_NBL0): now also RP905.7 (P7); no longer U301.39 (UDQM)
- net at U201.B12 (PD0/FMC_D2): now also RP901.3 (P3); no longer U301.5 (DQ2)
- net at U201.B7 (PG15/FMC_SDNCAS): now also RP905.4 (P4); no longer U301.17 (~CAS)
- net at U201.C12 (PD1/FMC_D3): now also RP901.4 (P4); no longer U301.7 (DQ3)
- net at U201.D2 (PF0/FMC_A0): now also RP903.1 (P1); no longer U301.23 (A0)
- net at U201.E2 (PF1/FMC_A1): now also RP903.2 (P2); no longer U301.24 (A1)
- net at U201.G2 (PF2/FMC_A2): now also RP903.3 (P3); no longer U301.25 (A2)
- net at U201.H14 (PG8/FMC_SDCLK): now also RP905.5 (P5); no longer U301.38 (CLK)
- net at U201.H2 (PF3/FMC_A3): now also RP903.4 (P4); no longer U301.26 (A3)
- net at U201.J2 (PF4/FMC_A4): now also RP903.5 (P5); no longer U301.29 (A4)
- net at U201.J3 (PH5/FMC_SDNWE): now also RP905.2 (P2); no longer U301.16 (~WE)
- net at U201.J4 (PH3/FMC_SDNE0): now also RP905.1 (P1); no longer U301.19 (~CS)
- net at U201.K13 (PD15/FMC_D1): now also RP901.2 (P2); no longer U301.4 (DQ1)
- net at U201.K15 (PD10/FMC_D15): now also RP902.8 (P8); no longer U301.53 (DQ15)
- net at U201.K3 (PF5/FMC_A5): now also RP903.6 (P6); no longer U301.30 (A5)
- net at U201.K4 (PH2/FMC_SOCKE0): now also RP905.6 (P6); no longer U301.37 (CKE)
- net at U201.L12 (PD14/FMC_D0): now also RP901.1 (P1); no longer U301.2 (DQ0)
- net at U201.L14 (PD9/FMC_D14): now also RP902.7 (P7); no longer U301.51 (DQ14)
- net at U201.L15 (PD8/FMC_D13): now also RP902.6 (P6); no longer U301.50 (DQ13)
- net at U201.M6 (PF12/FMC_A6): now also RP903.7 (P7); no longer U301.31 (A6)
- net at U201.M7 (PG1/FMC_A11): now also RP904.4 (P4); no longer U301.35 (A11)
- net at U201.M8 (PF15/FMC_A9): now also RP904.2 (P2); no longer U301.34 (A9)
- net at U201.N11 (PG5/FMC_A15/FMC_BA1): now also RP904.5 (P5); no longer U301.21 (BA1)
- net at U201.N12 (PG4/FMC_A14/FMC_BA0): now also RP904.6 (P6); no longer U301.20 (BA0)
- net at U201.N6 (PF13/FMC_A7): now also RP903.8 (P8); no longer U301.32 (A7)
- net at U201.N7 (PG0/FMC_A10): now also RP904.3 (P3); no longer U301.22 (A10)
- net at U201.N9 (PE8/FMC_D5): now also RP901.6 (P6); no longer U301.10 (DQ5)
- net at U201.P10 (PE11/FMC_D8): now also RP902.1 (P1); no longer U301.42 (DQ8)
- net at U201.P11 (PE14/FMC_D11): now also RP902.4 (P4); no longer U301.47 (DQ11)
- net at U201.P6 (PF14/FMC_A8): now also RP904.1 (P1); no longer U301.33 (A8)
- net at U201.P8 (PF11/FMC_SDNRAS): now also RP905.3 (P3); no longer U301.18 (~RAS)
- net at U201.P9 (PE9/FMC_D6): now also RP901.7 (P7); no longer U301.11 (DQ6)
- net at U201.R10 (PE12/FMC_D9): now also RP902.2 (P2); no longer U301.44 (DQ9)
- net at U201.R11 (PE15/FMC_D12): now also RP902.5 (P5); no longer U301.48 (DQ12)
- net at U201.R12 (PE13/FMC_D10): now also RP902.3 (P3); no longer U301.45 (DQ10)
- net at U201.R8 (PE7/FMC_D4): now also RP901.5 (P5); no longer U301.8 (DQ4)
- net at U201.R9 (PE10/FMC_D7): now also RP901.8 (P8); no longer U301.13 (DQ7)
- new net: RP901.11 (R6), U301.10 (DQ5)
- new net: RP901.10 (R7), U301.11 (DQ6)
- new net: RP901.9 (R8), U301.13 (DQ7)
- new net: RP905.9 (R8), U301.15 (LDQM)
- new net: RP905.15 (R2), U301.16 (~WE)
- new net: RP905.13 (R4), U301.17 (~CAS)
- new net: RP905.14 (R3), U301.18 (~RAS)
- new net: RP905.16 (R1), U301.19 (~CS)
- new net: RP901.16 (R1), U301.2 (DQ0)
- new net: RP904.11 (R6), U301.20 (BA0)
- new net: RP904.12 (R5), U301.21 (BA1)
- new net: RP904.14 (R3), U301.22 (A10)
- new net: RP903.16 (R1), U301.23 (A0)
- new net: RP903.15 (R2), U301.24 (A1)
- new net: RP903.14 (R3), U301.25 (A2)
- new net: RP903.13 (R4), U301.26 (A3)
- new net: RP903.12 (R5), U301.29 (A4)
- new net: RP903.11 (R6), U301.30 (A5)
- new net: RP903.10 (R7), U301.31 (A6)
- new net: RP903.9 (R8), U301.32 (A7)
- new net: RP904.16 (R1), U301.33 (A8)
- new net: RP904.15 (R2), U301.34 (A9)
- new net: RP904.13 (R4), U301.35 (A11)
- new net: RP905.11 (R6), U301.37 (CKE)
- new net: RP905.12 (R5), U301.38 (CLK)
- new net: RP905.10 (R7), U301.39 (UDQM)
- new net: RP901.15 (R2), U301.4 (DQ1)
- new net: RP902.16 (R1), U301.42 (DQ8)
- new net: RP902.15 (R2), U301.44 (DQ9)
- new net: RP902.14 (R3), U301.45 (DQ10)
- new net: RP902.13 (R4), U301.47 (DQ11)
- new net: RP902.12 (R5), U301.48 (DQ12)
- new net: RP901.14 (R3), U301.5 (DQ2)
- new net: RP902.11 (R6), U301.50 (DQ13)
- new net: RP902.10 (R7), U301.51 (DQ14)
- new net: RP902.9 (R8), U301.53 (DQ15)
- new net: RP901.13 (R4), U301.7 (DQ3)
- new net: RP901.12 (R5), U301.8 (DQ4)
Other:
- moved on the sheet: C301, C302, C303, C304, C305, C306, C307, U201P, U301

Commit message: Removed WiFi Module added Footprints
Parts:
- J901: footprint (none) -> Connectors_Hirose:microSD_Card_Receptacle_Hirose_DM3AT-SF-PEJM5
- U201: footprint (none) -> buttons:STM32F439NI
Changed lines of the file:
@@
 F 0 "U201" H 8450 2850 60  0000 L CNN
 F 1 "STM32F439NIH6" H 8450 2750 60  0000 L CNN
-F 2 "" H 8250 2600 60  0001 C CNN
+F 2 "buttons:STM32F439NI" H 8250 2600 60  0001 C CNN
 F 3 "" H 8250 2600 60  0000 C CNN
 	16   8250 2600
@@
 F 0 "U201" H 2350 1950 60  0000 L CNN
 F 1 "STM32F439NIH6" H 2350 1850 60  0000 L CNN
-F 2 "" H 2150 1400 60  0001 C CNN
+F 2 "buttons:STM32F439NI" H 2150 1400 60  0001 C CNN
 F 3 "" H 2150 1400 60  0000 C CNN
 	4    2150 1400
@@
 Connection ~ 5450 6000
 $Comp
-L GND #PWR095
+L GND #PWR0107
 U 1 1 584DBACB
 P 5450 6600
-F 0 "#PWR095" H 5450 6350 50  0001 C CNN
+F 0 "#PWR0107" H 5450 6350 50  0001 C CNN
 F 1 "GND" H 5450 6450 50  0000 C CNN
 F 2 "" H 5450 6600 50  0000 C CNN
@@
 Connection ~ 5450 6500
 $Comp
-L VCC #PWR096
+L VCC #PWR0108
 U 1 1 584DBB5F
 P 5450 5100
-F 0 "#PWR096" H 5450 4950 50  0001 C CNN
+F 0 "#PWR0108" H 5450 4950 50  0001 C CNN
 F 1 "VCC" H 5450 5250 50  0000 C CNN
 F 2 "" H 5450 5100 50  0000 C CNN
@@
 F 0 "J901" H 10350 3050 60  0000 C CNN
 F 1 "MICRO_SD" H 10300 3550 60  0000 C CNN
-F 2 "" V 10410 2500 60  0001 C CNN
+F 2 "Connectors_Hirose:microSD_Card_Receptacle_Hirose_DM3AT-SF-PEJM5" V 10410 2500 60  0001 C CNN
 F 3 "" V 10410 2500 60  0000 C CNN
 	1    10300 3000
@@
 $EndComp
 $Comp
-L GND #PWR097
+L GND #PWR0109
 U 1 1 584DD873
 P 10550 3800
-F 0 "#PWR097" H 10550 3550 50  0001 C CNN
+F 0 "#PWR0109" H 10550 3550 50  0001 C CNN
 F 1 "GND" H 10550 3650 50  0000 C CNN
 F 2 "" H 10550 3800 50  0000 C CNN
@@
 	8550 2600 8250 2600
 $Comp
-L +3V3 #PWR098
+L +3V3 #PWR0110
 U 1 1 584E0DE7
 P 9250 1800
-F 0 "#PWR098" H 9250 1650 50  0001 C CNN
+F 0 "#PWR0110" H 9250 1650 50  0001 C CNN
 F 1 "+3V3" H 9250 1940 50  0000 C CNN
 F 2 "" H 9250 1800 50  0000 C CNN
@@
 Connection ~ 8350 2800
 $Comp
-L GND #PWR099
+L GND #PWR0111
 U 1 1 584E1578
 P 8950 2250
-F 0 "#PWR099" H 8950 2000 50  0001 C CNN
+F 0 "#PWR0111" H 8950 2000 50  0001 C CNN
 F 1 "GND" H 8950 2100 50  0000 C CNN
 F 2 "" H 8950 2250 50  0000 C CNN
@@
 $EndComp
 $Comp
-L GND #PWR0100
+L GND #PWR0112
 U 1 1 584E15BF
 P 8650 2250
-F 0 "#PWR0100" H 8650 2000 50  0001 C CNN
+F 0 "#PWR0112" H 8650 2000 50  0001 C CNN
 F 1 "GND" H 8650 2100 50  0000 C CNN
 F 2 "" H 8650 2250 50  0000 C CNN
