File: MEMORY.sch (KiCad schematic (older format))
At the start: 36 parts, among them J901 MICRO_SD, U201 STM32F439NIH6, U301 IS42S16400J

Commit message: started working on implementing i.MX7 core into base schematic
Parts:
- removed C301, C302, C303, C304, C305, C306, C307, C904: 100n, Capacitors_SMD:C_0603, symbol C
- removed C903: 10u, Capacitors_SMD:C_0603, symbol C
- removed J901: MICRO_SD, Connectors_Hirose:microSD_Card_Receptacle_Hirose_DM3AT-SF-PEJM5, symbol MICRO_SD
- removed R910: 10k, Resistors_SMD:R_0603, symbol R
- removed R911, R912, R913, R915, R916: 10, Resistors_SMD:R_0603, symbol R
- removed R914: 22, Resistors_SMD:R_0603, symbol R
- removed RP901, RP902, RP903, RP904, RP905: 100, Resistors_SMD:R_Array_Convex_8x0602, symbol R_PACK8
- removed TP901, TP902, TP903, TP904, TP905, TP906, TP907, TP908, TP909, TP910, TP911, TP912: TP, buttons:TP, symbol TP
- removed U201: STM32F439NIH6, buttons:STM32F439NI, symbol STM32F439NIH6
- removed U301: IS42S16400J, symbol IS42S16400J
- added C?: 100n, symbol C
- added C? (x34): 220n, symbol C
- added C? (x5): 22u, symbol C
- added J? (x24): GND, symbol TEST_1P
- added R? (x3): 0R, symbol R
- added R? (x3): 240R, symbol R
- added R? (x2): 10k, symbol R
- added R? (x2): 470R, symbol R
- added U2: MCIMX7D7DVM10SC, symbol MCIMX7D7DVM10SC
- added U? (x2): MT41K256M16HA-125, symbol MT41K256M16HA-125
Connections:
- net labels added: CAS, CS0, CS1, DDR_VREF, DQM0, DQM1, DQM2, DQM3, DRAM_ADDR0, DRAM_ADDR1, DRAM_ADDR10, DRAM_ADDR11, DRAM_ADDR12, DRAM_ADDR13, DRAM_ADDR14, DRAM_ADDR15, DRAM_ADDR2, DRAM_ADDR3, DRAM_ADDR4, DRAM_ADDR5, DRAM_ADDR6, DRAM_ADDR7, DRAM_ADDR8, DRAM_ADDR9, DRAM_ADDR[0..14], DRAM_DATA0, DRAM_DATA1, DRAM_DATA10, DRAM_DATA11, DRAM_DATA12, DRAM_DATA13, DRAM_DATA14, DRAM_DATA15, DRAM_DATA16, DRAM_DATA17, DRAM_DATA18, DRAM_DATA19, DRAM_DATA2, DRAM_DATA20, DRAM_DATA21, DRAM_DATA22, DRAM_DATA23, DRAM_DATA24, DRAM_DATA25, DRAM_DATA26, DRAM_DATA27, DRAM_DATA28, DRAM_DATA29, DRAM_DATA3, DRAM_DATA30, DRAM_DATA31, DRAM_DATA4, DRAM_DATA5, DRAM_DATA6, DRAM_DATA7, DRAM_DATA8, DRAM_DATA9, DRAM_DATA[0..31], DRAM_ZQ, NVCC_DRAM, NVCC_DRAM_CKE, ODT0, ODT1, RAS, RESET, SDBA0, SDBA1, SDBA2, SDCKE0, SDCKE1, SDCLK0_N, SDCLK0_P, SDQS0_N, SDQS0_P, SDQS1_N, SDQS1_P, SDQS2_N, SDQS2_P, SDQS3_N, SDQS3_P, SDWE, VDD_VREF
- net labels removed: +3V3, VCC
- wire segments 188 -> 398
- no-connect marks 18 -> 0
Other:
- note added: "Place left points to CPU and \nright points to RAM\nfor signal integrity measurement"
- note added: "Place near BANK0"
- note added: "Place near BANK1"
- note added: "Place near CPU"
- note removed: "place caps close to SDRAM"

Commit message: modified adui circuit
Changed lines of the file:
@@
 LIBS:mtfc8gacaeam-1m_wt
 LIBS:sn74avc2t244
-LIBS:lsm9ds1
+LIBS:WM8960CGEFL
 LIBS:3210retro-cache
 EELAYER 25 0
@@
 Wire Bus Line
 	6600 1350 6600 4000
-Text Label 1800 800  0    60   ~ 0
+Text Label 1700 1100 0    60   ~ 0
 DRAM_DATA[0..31]
 Text Label 5600 1350 0    60   ~ 0
