File: MEMORY.sch (KiCad schematic (older format))
At the start: 77 parts, among them J901 GND, J902 GND, J903 GND, J904 GND, J905 GND, J906 GND, J907 GND, J908 GND, J909 GND, J910 GND, J911 GND, J912 GND, J913 GND, J914 GND, J915 GND, J916 GND, J917 GND, J918 GND, J919 GND, J920 GND, J921 GND, J922 GND, J923 GND, J924 GND, U801 MCIMX7D7DVM10SC, U901 MT41K256M16HA-125, U902 MT41K256M16HA-125

Commit message: added footprint for RAM, annotated sheets again
Parts:
- U901, U902: footprint NokiaRetroFit:MT41K256M16HA-125 -> NokiaRetroFit:FBGA_96_x16
Changed lines of the file:
@@
-	1    0    0    -1
-$EndComp
-$Comp
-L MT41K256M16HA-125 U902
-U 1 1 590B6323
-P 13500 2700
-F 0 "U902" H 14550 3150 60  0000 C CNN
-F 1 "MT41K256M16HA-125" H 13500 2700 60  0000 C CNN
-F 2 "NokiaRetroFit:MT41K256M16HA-125" H 13500 2700 60  0001 C CNN
-F 3 "" H 13500 2700 60  0001 C CNN
-	1    13500 2700
 	1    0    0    -1
 $EndComp
@@
 DQM3
 $Comp
-L NVCC_DRAM #PWR0164
+L NVCC_DRAM #PWR901
 U 1 1 591D8B55
 P 2200 6800
-F 0 "#PWR0164" H 2200 6650 50  0001 C CNN
+F 0 "#PWR901" H 2200 6650 50  0001 C CNN
 F 1 "NVCC_DRAM" H 2200 6950 50  0000 C CNN
 F 2 "" H 2200 6800 50  0001 C CNN
@@
 	6500 7300 6500 7200
 $Comp
-L NVCC_DRAM #PWR0165
+L NVCC_DRAM #PWR911
 U 1 1 591D9FCD
 P 6500 7200
-F 0 "#PWR0165" H 6500 7050 50  0001 C CNN
+F 0 "#PWR911" H 6500 7050 50  0001 C CNN
 F 1 "NVCC_DRAM" H 6500 7350 50  0000 C CNN
 F 2 "" H 6500 7200 50  0001 C CNN
@@
 $EndComp
 $Comp
-L GND #PWR0166
+L GND #PWR904
 U 1 1 591DA1AD
 P 5350 8350
-F 0 "#PWR0166" H 5350 8100 50  0001 C CNN
+F 0 "#PWR904" H 5350 8100 50  0001 C CNN
 F 1 "GND" H 5350 8200 50  0000 C CNN
 F 2 "" H 5350 8350 50  0001 C CNN
@@
 $EndComp
 $Comp
-L GND #PWR0167
+L GND #PWR905
 U 1 1 591DA1D4
 P 5650 8350
-F 0 "#PWR0167" H 5650 8100 50  0001 C CNN
+F 0 "#PWR905" H 5650 8100 50  0001 C CNN
 F 1 "GND" H 5650 8200 50  0000 C CNN
 F 2 "" H 5650 8350 50  0001 C CNN
@@
 $EndComp
 $Comp
-L GND #PWR0168
+L GND #PWR906
 U 1 1 591DA1F4
 P 5950 8350
-F 0 "#PWR0168" H 5950 8100 50  0001 C CNN
+F 0 "#PWR906" H 5950 8100 50  0001 C CNN
 F 1 "GND" H 5950 8200 50  0000 C CNN
 F 2 "" H 5950 8350 50  0001 C CNN
@@
 DQM0
 $Comp
-L VDD_VREF #PWR0169
+L VDD_VREF #PWR909
 U 1 1 591DA9C3
 P 6500 6050
-F 0 "#PWR0169" H 6500 5900 50  0001 C CNN
+F 0 "#PWR909" H 6500 5900 50  0001 C CNN
 F 1 "VDD_VREF" H 6500 6200 50  0000 C CNN
 F 2 "" H 6500 6050 50  0001 C CNN
@@
 Connection ~ 7300 6100
 $Comp
-L GND #PWR0170
+L GND #PWR910
 U 1 1 591DAF04
 P 6500 6500
-F 0 "#PWR0170" H 6500 6250 50  0001 C CNN
+F 0 "#PWR910" H 6500 6250 50  0001 C CNN
 F 1 "GND" H 6500 6350 50  0000 C CNN
 F 2 "" H 6500 6500 50  0001 C CNN
@@
 	6500 6500 6500 6450
 $Comp
-L GND #PWR0171
+L GND #PWR912
 U 1 1 591DAF31
 P 6800 6500
-F 0 "#PWR0171" H 6800 6250 50  0001 C CNN
+F 0 "#PWR912" H 6800 6250 50  0001 C CNN
 F 1 "GND" H 6800 6350 50  0000 C CNN
 F 2 "" H 6800 6500 50  0001 C CNN
@@
 	6800 6500 6800 6450
 $Comp
-L GND #PWR0172
+L GND #PWR917
 U 1 1 591DB057
 P 7300 6900
-F 0 "#PWR0172" H 7300 6650 50  0001 C CNN
+F 0 "#PWR917" H 7300 6650 50  0001 C CNN
 F 1 "GND" H 7300 6750 50  0000 C CNN
 F 2 "" H 7300 6900 50  0001 C CNN
@@
 	7300 6400 7300 6500
 $Comp
-L GND #PWR0173
+L GND #PWR918
 U 1 1 591DB3A1
 P 7700 7100
-F 0 "#PWR0173" H 7700 6850 50  0001 C CNN
+F 0 "#PWR918" H 7700 6850 50  0001 C CNN
 F 1 "GND" H 7700 6950 50  0000 C CNN
 F 2 "" H 7700 7100 50  0001 C CNN
@@
 SDQS2_N
 $Comp
-L GND #PWR0174
+L GND #PWR927
 U 1 1 591DD3B2
 P 12050 6900
-F 0 "#PWR0174" H 12050 6650 50  0001 C CNN
+F 0 "#PWR927" H 12050 6650 50  0001 C CNN
 F 1 "GND" H 12050 6750 50  0000 C CNN
 F 2 "" H 12050 6900 50  0001 C CNN
@@
 $EndComp
 $Comp
-L GND #PWR0175
+L GND #PWR928
 U 1 1 591DD3B8
 P 12450 7100
-F 0 "#PWR0175" H 12450 6850 50  0001 C CNN
+F 0 "#PWR928" H 12450 6850 50  0001 C CNN
 F 1 "GND" H 12450 6950 50  0000 C CNN
 F 2 "" H 12450 7100 50  0001 C CNN
@@
 	12050 6400 12050 6500
 $Comp
-L VDD_VREF #PWR0176
+L VDD_VREF #PWR924
 U 1 1 591DD5A2
 P 11250 6050
-F 0 "#PWR0176" H 11250 5900 50  0001 C CNN
+F 0 "#PWR924" H 11250 5900 50  0001 C CNN
 F 1 "VDD_VREF" H 11250 6200 50  0000 C CNN
 F 2 "" H 11250 6050 50  0001 C CNN
@@
 Connection ~ 11550 6100
 $Comp
-L GND #PWR0177
+L GND #PWR925
 U 1 1 591DD5B9
 P 11250 6500
-F 0 "#PWR0177" H 11250 6250 50  0001 C CNN
+F 0 "#PWR925" H 11250 6250 50  0001 C CNN
 F 1 "GND" H 11250 6350 50  0000 C CNN
 F 2 "" H 11250 6500 50  0001 C CNN
@@
 	11250 6500 11250 6450
 $Comp
-L GND #PWR0178
+L GND #PWR926
 U 1 1 591DD5C0
 P 11550 6500
-F 0 "#PWR0178" H 11550 6250 50  0001 C CNN
+F 0 "#PWR926" H 11550 6250 50  0001 C CNN
 F 1 "GND" H 11550 6350 50  0000 C CNN
 F 2 "" H 11550 6500 50  0001 C CNN
@@
 Connection ~ 8150 1900
 $Comp
-L NVCC_DRAM #PWR0179
+L NVCC_DRAM #PWR929
 U 1 1 591DF650
 P 12600 1850
-F 0 "#PWR0179" H 12600 1700 50  0001 C CNN
+F 0 "#PWR929" H 12600 1700 50  0001 C CNN
 F 1 "NVCC_DRAM" H 12600 2000 50  0000 C CNN
 F 2 "" H 12600 1850 50  0001 C CNN
@@
 	11500 5300 11500 5200
 $Comp
-L GND #PWR0180
+L GND #PWR908
 U 1 1 591E04B8
 P 6000 6900
-F 0 "#PWR0180" H 6000 6650 50  0001 C CNN
+F 0 "#PWR908" H 6000 6650 50  0001 C CNN
 F 1 "GND" H 6000 6750 50  0000 C CNN
 F 2 "" H 6000 6900 50  0001 C CNN
@@
 $EndComp
 $Comp
-L GND #PWR0181
+L GND #PWR907
 U 1 1 591E355B
 P 6000 6100
-F 0 "#PWR0181" H 6000 5850 50  0001 C CNN
+F 0 "#PWR907" H 6000 5850 50  0001 C CNN
 F 1 "GND" H 6000 5950 50  0000 C CNN
 F 2 "" H 6000 6100 50  0001 C CNN
@@
 $EndComp
 $Comp
-L NVCC_DRAM #PWR0182
+L NVCC_DRAM #PWR902
 U 1 1 591E38C2
 P 2900 9400
-F 0 "#PWR0182" H 2900 9250 50  0001 C CNN
+F 0 "#PWR902" H 2900 9250 50  0001 C CNN
 F 1 "NVCC_DRAM" H 2900 9550 50  0000 C CNN
 F 2 "" H 2900 9400 50  0001 C CNN
@@
 	4400 9850 4400 9800
 $Comp
-L GND #PWR0183
+L GND #PWR903
 U 1 1 591E4185
 P 2900 9900
-F 0 "#PWR0183" H 2900 9650 50  0001 C CNN
+F 0 "#PWR903" H 2900 9650 50  0001 C CNN
 F 1 "GND" H 2900 9750 50  0000 C CNN
 F 2 "" H 2900 9900 50  0001 C CNN
@@
 $EndComp
 $Comp
-L NVCC_DRAM #PWR0184
+L NVCC_DRAM #PWR913
 U 1 1 591E46CB
 P 7050 8450
-F 0 "#PWR0184" H 7050 8300 50  0001 C CNN
+F 0 "#PWR913" H 7050 8300 50  0001 C CNN
 F 1 "NVCC_DRAM" H 7050 8600 50  0000 C CNN
 F 2 "" H 7050 8450 50  0001 C CNN
@@
 	8850 8900 8850 8850
 $Comp
-L GND #PWR0185
+L GND #PWR914
 U 1 1 591E46FE
 P 7050 8950
-F 0 "#PWR0185" H 7050 8700 50  0001 C CNN
+F 0 "#PWR914" H 7050 8700 50  0001 C CNN
 F 1 "GND" H 7050 8800 50  0000 C CNN
 F 2 "" H 7050 8950 50  0001 C CNN
@@
 $EndComp
 $Comp
-L NVCC_DRAM #PWR0186
+L NVCC_DRAM #PWR915
 U 1 1 591E4F77
 P 7050 9400
-F 0 "#PWR0186" H 7050 9250 50  0001 C CNN
+F 0 "#PWR915" H 7050 9250 50  0001 C CNN
 F 1 "NVCC_DRAM" H 7050 9550 50  0000 C CNN
 F 2 "" H 7050 9400 50  0001 C CNN
@@
 	8850 9850 8850 9800
 $Comp
-L GND #PWR0187
+L GND #PWR916
 U 1 1 591E4FAA
 P 7050 9900
-F 0 "#PWR0187" H 7050 9650 50  0001 C CNN
+F 0 "#PWR916" H 7050 9650 50  0001 C CNN
 F 1 "GND" H 7050 9750 50  0000 C CNN
 F 2 "" H 7050 9900 50  0001 C CNN
@@
 $EndComp
 $Comp
-L NVCC_DRAM #PWR0188
+L NVCC_DRAM #PWR920
 U 1 1 591E6BFA
 P 9550 8450
-F 0 "#PWR0188" H 9550 8300 50  0001 C CNN
+F 0 "#PWR920" H 9550 8300 50  0001 C CNN
 F 1 "NVCC_DRAM" H 9550 8600 50  0000 C CNN
 F 2 "" H 9550 8450 50  0001 C CNN
@@
 	11350 8900 11350 8850
 $Comp
-L GND #PWR0189
+L GND #PWR921
 U 1 1 591E6C39
 P 9550 8950
-F 0 "#PWR0189" H 9550 8700 50  0001 C CNN
+F 0 "#PWR921" H 9550 8700 50  0001 C CNN
 F 1 "GND" H 9550 8800 50  0000 C CNN
 F 2 "" H 9550 8950 50  0001 C CNN
@@
 $EndComp
 $Comp
-L NVCC_DRAM #PWR0190
+L NVCC_DRAM #PWR922
 U 1 1 591E6C59
 P 9550 9400
-F 0 "#PWR0190" H 9550 9250 50  0001 C CNN
+F 0 "#PWR922" H 9550 9250 50  0001 C CNN
 F 1 "NVCC_DRAM" H 9550 9550 50  0000 C CNN
 F 2 "" H 9550 9400 50  0001 C CNN
@@
 	11350 9850 11350 9800
 $Comp
-L GND #PWR0191
+L GND #PWR923
 U 1 1 591E6C98
 P 9550 9900
-F 0 "#PWR0191" H 9550 9650 50  0001 C CNN
+F 0 "#PWR923" H 9550 9650 50  0001 C CNN
 F 1 "GND" H 9550 9750 50  0000 C CNN
 F 2 "" H 9550 9900 50  0001 C CNN
@@
 	7850 1850 7850 2100
 $Comp
-L NVCC_DRAM #PWR0192
+L NVCC_DRAM #PWR919
 U 1 1 591DDA84
 P 7850 1850
-F 0 "#PWR0192" H 7850 1700 50  0001 C CNN
+F 0 "#PWR919" H 7850 1700 50  0001 C CNN
 F 1 "NVCC_DRAM" H 7850 2000 50  0000 C CNN
 F 2 "" H 7850 1850 50  0001 C CNN
@@
 $EndComp
 $Comp
+L MT41K256M16HA-125 U902
+U 1 1 59770762
+P 13500 2700
+F 0 "U902" H 14550 3150 60  0000 C CNN
+F 1 "MT41K256M16HA-125" H 13500 2700 60  0000 C CNN
+F 2 "NokiaRetroFit:FBGA_96_x16" H 13500 2700 60  0001 C CNN
+F 3 "" H 13500 2700 60  0001 C CNN
+	1    13500 2700
+	1    0    0    -1
+$EndComp
+$Comp
 L MT41K256M16HA-125 U901
-U 1 1 593FF3D0
+U 1 1 59770833
 P 8750 2700
 F 0 "U901" H 9800 3150 60  0000 C CNN
 F 1 "MT41K256M16HA-125" H 8750 2700 60  0000 C CNN
-F 2 "NokiaRetroFit:MT41K256M16HA-125" H 8750 2700 60  0001 C CNN
+F 2 "NokiaRetroFit:FBGA_96_x16" H 8750 2700 60  0001 C CNN
 F 3 "" H 8750 2700 60  0001 C CNN
 	1    8750 2700
