File: MCU.sch (KiCad schematic (older format))
At the start: 115 parts, among them P801 JTAG, Q201 BC817-40, U201 STM32F439NIH6, Y201 32kHz, Y202 24MHz

Commit message: Removed WiFi Module added Footprints
Parts:
- U201: footprint (none) -> buttons:STM32F439NI
- Y201, Y202: footprint (none) -> Crystals:Crystal_SMD_SeikoEpson_MC146-4pin_6.7x1.5mm_HandSoldering
Connections:
- net labels removed: BT[0..7], BT_EN, ESP_UART2, EXT_32K, WLAN_EN, WL[0..6]
- wire segments 170 -> 159
Other:
- moved on the sheet: R223, R224, TP813

Commit message: started working on implementing i.MX7 core into base schematic
Parts:
- removed Q201: BC817-40, TO_SOT_Packages_SMD:SOT-23, symbol BC817-40
- removed R201, R202, R203, R204, R205, R206: 10, Resistors_SMD:R_0603, symbol R
- removed R207, R208, R211, R212, R213, R214, R215, R216, R217, R218, R219, R220, R221, R222, R228, R229, R234, R235, R236, R237, R238, R239, R240, R241, R242, R243, R244, R245, R246, R247, R248, R816, R817, R818: 100, Resistors_SMD:R_0603, symbol R
- removed R209, R210, R227: 10k, Resistors_SMD:R_0603, symbol R
- removed R223, R224: R, Resistors_SMD:R_0603, symbol R
- removed TP801, TP802, TP803, TP804, TP805, TP806, TP807, TP808, TP809, TP810, TP812, TP813, TP814, TP815, TP816, TP817, TP818, TP819, TP820, TP821, TP822, TP823, TP824, TP825, TP826, TP827, TP828, TP829, TP830, TP831, TP832, TP833, TP834, TP835, TP836, TP837, TP838, TP839, TP840, TP841, TP842, TP843, TP844, TP845, TP846, TP847, TP848, TP849, TP850, TP851, TP852, TP853, TP854, TP855, TP856: TP, buttons:TP, symbol TP
- removed U201: STM32F439NIH6, buttons:STM32F439NI, symbol STM32F439NIH6
- added C?: 220n, Capacitors_SMD:C_0603, symbol C
- added C?: 100n, symbol C
- added D?: D_Schottky, symbol D_Schottky
- added R?: 47k, symbol R
- added R? (x2): 1k, symbol R
- added R? (x2): 0, symbol R
- added R? (x4): 10k, Resistors_SMD:R_0603, symbol R
- added R?: 4k7, Resistors_SMD:R_0603, symbol R
- added U?: MCIMX7D7DVM10SC, symbol MCIMX7D7DVM10SC
Connections:
- net labels added: VLDO3_3V3, VSNVS, ~POR
- net labels removed: +5V, DISPLAY_DATA0, DISPLAY_DATA1, DISPLAY_DATA10, DISPLAY_DATA11, DISPLAY_DATA12, DISPLAY_DATA13, DISPLAY_DATA14, DISPLAY_DATA15, DISPLAY_DATA16, DISPLAY_DATA2, DISPLAY_DATA3, DISPLAY_DATA4, DISPLAY_DATA5, DISPLAY_DATA6, DISPLAY_DATA7, DISPLAY_DATA8, DISPLAY_DATA9, DISPLAY_DATA[0..16], ESP_UART0, ESP_UART1, ESP_UART3, ESP_UART[0..3], VCC
- wire segments 159 -> 90
- no-connect marks 7 -> 15
Other:
- note added: "1GB DDR3 RAM"
- note removed: "SDRAM\n\nSD Card"
- moved on the sheet: C201, C202, C203, C204, P801, R815, TP811, Y201, Y202

Commit message: fixed message telling to rescue PF3000 symbol while opening the schematic
Changed lines of the file:
@@
 EESchema Schematic File Version 2
-LIBS:3210retro-rescue
 LIBS:power
 LIBS:device
@@
 	5300 7550 6200 7550
 Wire Wire Line
-	6200 6800 6200 7550
-Wire Wire Line
-	1250 6800 6200 6800
+	6200 7550 6200 6800
+Wire Wire Line
+	6200 6800 1250 6800
 Connection ~ 5750 6800
 $Comp

Commit message: Put key matrix into schematic. Using Keypad Peripheral of i.MX7
Parts:
- added U? (x2): MCIMX7D7DVM10SC, symbol MCIMX7D7DVM10SC
Connections:
- net labels added: KEYPAD_COL0, KEYPAD_COL1, KEYPAD_COL2, KEYPAD_COL3, KEYPAD_COL[0..3], KEYPAD_ROW0, KEYPAD_ROW1, KEYPAD_ROW2, KEYPAD_ROW3, KEYPAD_ROW[0..3], LED_PWM
- net labels removed: KEY0, KEY1, KEY2, KEY3, KEY4, KEY5, KEY6, KEY7, KEY[0..7], LED0, LED1, LED2, LED3, LED4, LED5, LED[0..5]
- wire segments 90 -> 93
Changed lines of the file:
@@
 LIBS:pf3000
 LIBS:voltages
-LIBS:3210retro-cache
-EELAYER 26 0
+EELAYER 25 0
 EELAYER END
 $Descr A3 16535 11693
@@
 Comment4 ""
 $EndDescr
-Text HLabel 8350 3400 0    60   BiDi ~ 0
-KEY[0..7]
+Text HLabel 15050 650  2    60   Input ~ 0
+KEYPAD_ROW[0..3]
 Text HLabel 1250 6800 0    60   Input ~ 0
 ~ON
@@
 $EndComp
 Wire Wire Line
-	8750 3700 9250 3700
-Wire Wire Line
-	8750 3800 9250 3800
-Wire Wire Line
-	8550 3900 9250 3900
-Wire Wire Line
-	8550 4000 9250 4000
-Wire Wire Line
-	8550 4100 9250 4100
-Wire Wire Line
-	8550 4200 9250 4200
-Wire Wire Line
-	8750 4500 9250 4500
-Wire Wire Line
-	8750 4600 9250 4600
-Wire Wire Line
-	8750 4700 9250 4700
-Wire Wire Line
-	8750 4800 9250 4800
-Wire Wire Line
-	8750 4900 9250 4900
-Wire Wire Line
-	8750 5000 9250 5000
-Wire Wire Line
-	8550 5100 9250 5100
-Wire Wire Line
-	8550 5200 9250 5200
+	13700 6050 14400 6050
+Wire Wire Line
+	13700 5850 14400 5850
+Wire Wire Line
+	13700 5650 14400 5650
+Wire Wire Line
+	13700 5450 14400 5450
+Wire Wire Line
+	13700 5950 14400 5950
+Wire Wire Line
+	13700 5750 14400 5750
+Wire Wire Line
+	13700 5550 14400 5550
+Wire Wire Line
+	13700 5350 14400 5350
 $Comp
 L Crystal Y202
@@
 $EndComp
 Wire Bus Line
-	8650 3400 8650 4900
-Entry Wire Line
-	8650 4400 8750 4500
-Entry Wire Line
-	8650 4500 8750 4600
-Entry Wire Line
-	8650 4600 8750 4700
-Entry Wire Line
-	8650 4700 8750 4800
-Entry Wire Line
-	8650 4800 8750 4900
-Entry Wire Line
-	8650 4900 8750 5000
-Entry Wire Line
-	8450 5000 8550 5100
-Entry Wire Line
-	8450 5100 8550 5200
-Wire Bus Line
-	8650 3400 8350 3400
-Entry Wire Line
-	8650 3600 8750 3700
-Entry Wire Line
-	8650 3700 8750 3800
-Text Label 8800 3700 0    60   ~ 0
-KEY0
-Text Label 8800 3800 0    60   ~ 0
-KEY1
-Text Label 8800 4500 0    60   ~ 0
-KEY2
-Text Label 8800 4600 0    60   ~ 0
-KEY3
-Text Label 8800 4700 0    60   ~ 0
-KEY4
-Text Label 8800 4800 0    60   ~ 0
-KEY5
-Text Label 8800 4900 0    60   ~ 0
-KEY6
-Text Label 8800 5000 0    60   ~ 0
-KEY7
-Text HLabel 8350 3550 0    60   Output ~ 0
-LED[0..5]
-Wire Bus Line
-	8350 3550 8450 3550
-Wire Bus Line
-	8450 3550 8450 5100
-Entry Wire Line
-	8450 3800 8550 3900
-Entry Wire Line
-	8450 3900 8550 4000
-Entry Wire Line
-	8450 4000 8550 4100
-Entry Wire Line
-	8450 4100 8550 4200
-Text Label 8800 5100 0    60   ~ 0
-LED0
-Text Label 8800 5200 0    60   ~ 0
-LED1
-Text Label 8800 3900 0    60   ~ 0
-LED2
-Text Label 8800 4000 0    60   ~ 0
-LED3
-Text Label 8800 4100 0    60   ~ 0
-LED4
-Text Label 8800 4200 0    60   ~ 0
-LED5
+	13850 650  13950 650
+Text Label 14400 6050 2    60   ~ 0
+KEYPAD_COL0
+Text Label 14400 5850 2    60   ~ 0
+KEYPAD_COL1
+Text Label 14400 5650 2    60   ~ 0
+KEYPAD_COL2
+Text Label 14400 5450 2    60   ~ 0
+KEYPAD_COL3
+Text Label 14400 5950 2    60   ~ 0
+KEYPAD_ROW0
+Text Label 14400 5750 2    60   ~ 0
+KEYPAD_ROW1
+Text Label 14400 5550 2    60   ~ 0
+KEYPAD_ROW2
+Text Label 14400 5350 2    60   ~ 0
+KEYPAD_ROW3
+Text HLabel 4650 4350 2    60   Output ~ 0
+LED_PWM
 Entry Wire Line
 	7950 850  8050 750
@@
 	5300 7550 6200 7550
 Wire Wire Line
-	6200 7550 6200 6800
-Wire Wire Line
-	6200 6800 1250 6800
+	6200 6800 6200 7550
+Wire Wire Line
+	1250 6800 6200 6800
 Connection ~ 5750 6800
 $Comp
@@
 Connection ~ 2500 7150
 Connection ~ 2800 7550
+$Comp
+L MCIMX7D7DVM10SC U?
+U 8 1 594174AE
+P 12600 1800
+F 0 "U?" H 12600 1800 60  0000 L CNN
+F 1 "MCIMX7D7DVM10SC" H 12600 1700 60  0000 L CNN
+F 2 "" H 10350 3500 60  0001 C CNN
+F 3 "" H 10350 3500 60  0001 C CNN
+	8    12600 1800
+	1    0    0    -1
+$EndComp
+Text HLabel 13950 650  2    60   Output ~ 0
+KEYPAD_COL[0..3]
+Wire Bus Line
+	19050 5200 19050 5200
+Wire Wire Line
+	13750 1150 13050 1150
+Wire Wire Line
+	13750 1050 13050 1050
+Wire Wire Line
+	13750 950  13050 950
+Wire Wire Line
+	13750 850  13050 850
+Wire Wire Line
+	14850 1150 14150 1150
+Wire Wire Line
+	14850 1050 14150 1050
+Wire Wire Line
+	14850 950  14150 950
+Wire Wire Line
+	14850 850  14150 850
+Text Label 13050 1150 0    60   ~ 0
+KEYPAD_COL0
+Text Label 13050 1050 0    60   ~ 0
+KEYPAD_COL1
+Text Label 13050 950  0    60   ~ 0
+KEYPAD_COL2
+Text Label 13050 850  0    60   ~ 0
+KEYPAD_COL3
+Text Label 14150 1150 0    60   ~ 0
+KEYPAD_ROW0
+Text Label 14150 1050 0    60   ~ 0
+KEYPAD_ROW1
+Text Label 14150 950  0    60   ~ 0
+KEYPAD_ROW2
+Text Label 14150 850  0    60   ~ 0
+KEYPAD_ROW3
+Wire Bus Line
+	15050 650  14950 650
+Wire Bus Line
+	14950 650  14950 1050
+Entry Wire Line
+	14850 850  14950 750
+Entry Wire Line
+	14850 950  14950 850
+Entry Wire Line
+	14850 1050 14950 950
+Entry Wire Line
+	14850 1150 14950 1050
+Wire Bus Line
+	13850 650  13850 1050
+Entry Wire Line
+	13750 1150 13850 1050
+Entry Wire Line
+	13750 1050 13850 950
+Entry Wire Line
+	13750 950  13850 850
+Entry Wire Line
+	13750 850  13850 750
+$Comp
+L MCIMX7D7DVM10SC U?
+U 6 1 5941FF2F
+P 2300 3800
+F 0 "U?" H 2300 3800 60  0000 L CNN
+F 1 "MCIMX7D7DVM10SC" H 2300 3700 60  0000 L CNN
+F 2 "" H 50  5500 60  0001 C CNN
+F 3 "" H 50  5500 60  0001 C CNN
+	6    2300 3800
+	1    0    0    -1
+$EndComp
+Wire Wire Line
+	4650 4350 3400 4350
 $EndSCHEMATC

Commit message: Added SD card, eMMC, Display
Parts:
- added C? (x2): 220n, symbol C
- added C?: 22u, symbol C
- added C? (x3): 2u2, symbol C
- added C? (x2): 470n, symbol C
- added L?: 100R, Resistors_SMD:R_0603, symbol L_Small
- added R?: 100k, symbol R
- added R?: 0, symbol R
- added U?: MCIMX7D7DVM10SC, symbol MCIMX7D7DVM10SC
Connections:
- net labels added: LCD_CLK, LCD_DATA00, LCD_DATA01, LCD_DATA02, LCD_DATA03, LCD_DATA04, LCD_DATA05, LCD_DATA06, LCD_DATA07, LCD_DATA08, LCD_DATA09, LCD_DATA10, LCD_DATA11, LCD_DATA12, LCD_DATA13, LCD_DATA14, LCD_DATA15, LCD_DATA16, LCD_DATA17, LCD_DATA18, LCD_DATA19, LCD_DATA20, LCD_DATA21, LCD_DATA22, LCD_DATA23, LCD_DATA[0..23], LCD_ENABLE, LCD_HSYNC, LCD_RESET, LCD_VSYNC, NVCC_3V3, PWM1_OUT, PWM2_OUT, PWM3_OUT, PWM4_OUT, RUMBLE_PWM, SAI1[0..6], SAI2[0..3], SW2OUT
- wire segments 93 -> 166
Other:
- note added: "uSD-Card Slot\n8GB eMMC"
- moved on the sheet: C205, C206, R225, R226

Commit message: Connected WIFI subsheet with ESP8266 and WL1807MOD to SD2 Connected WL1807MOD Bluetoth UART to UART3 Connected A7 Module AT UART to UART6 Connected A7 GPS UART to UART5 Connected A7 HS download to UART7 Connected debug pins to UART1 Connected debug pins to UART2 Added CPU_PWR subsheet to connect power rails to i.MX7 A7 UARTs are routed through level shifter to get from 2.8V to 3.3V All the sheets should be on A3 size now Externel USB is connected to USB_OTG1 Board power sheet is cleared out. Only 4V booster is needed.
Parts:
- removed C205, C206: C, Capacitors_SMD:C_0603, symbol C
- removed R225, R226: 100, Resistors_SMD:R_0603, symbol R
- added C? (x2): 470n, symbol C
- added C?: 10u, symbol C
- added P?: A7, symbol CONN_01X02
- added P?: M4, symbol CONN_01X02
- added R?: 200R, symbol R
- added U? (x2): MCIMX7D7DVM10SC, symbol MCIMX7D7DVM10SC
Connections:
- net labels added: AT_UART0, AT_UART1, AT_UART2, AT_UART3, AT_UART[0..3], AT_UART_CTS, AT_UART_RTS, AT_UART_RX, AT_UART_TX, BT0, BT1, BT2, BT3, BT[0..7], BT_EN, BT_UART_CTS, BT_UART_RTS, BT_UART_RX, BT_UART_TX, GPIO2_D10, GPIO2_D11, GPIO2_D9, NVCC_1V8, SD2_BUS[0..8], SWBSTOUT, UART6_RX, UART7_CTS, UART7_RTS, UART7_RX, UART7_TX, VDDA
- net labels removed: 1V8_ref, 3V3_PG, 3V3_ref, 4V_ref, CH_PD, GPIO0, GPIO12, GPIO13, RESET, UART0, UART1, UART2, UART3, UART[0..3], ~INT, ~LINK_UP
- wire segments 166 -> 190
- no-connect marks 15 -> 18
Other:
- moved on the sheet: C?, U?H

Commit message: Moved USB into it's own subsheet shuffeld stuff around to make it less crammed
Parts:
- removed C?: 10u, symbol C
- removed R?: 200R, symbol R
- removed U?: MCIMX7D7DVM10SC, symbol MCIMX7D7DVM10SC
Connections:
- net labels added: UART5_RX
- net labels removed: SWBSTOUT, UART6_RX
- wire segments 190 -> 212
- no-connect marks 18 -> 16
Other:
- note removed: "50Ohm"
- moved on the sheet: C201, C202, C203, C204, C?, D?, P801, P?, R815, R?, TP811, U?B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

Commit message: renamed USB.sch to USB_IMU.sch added LSM9DS1 IMU to USB_IMU.sch and connected I2C2 bus shuffeld stuff around to make MCU.sch less crammed
Parts:
- added C?: 470n, symbol C
Connections:
- net labels added: I2C1_SCL, I2C1_SDA, PMIC_SD_CSEL
- wire segments 212 -> 201
Other:
- moved on the sheet: C?, L?, P?, R?, U?A, U?G
