File: STORAGE.sch (KiCad schematic (older format))
At the start: 10 parts, among them J1101 MICRO_SD_HINGE, U1101 MTFC8GACAEAM-1M_WT, U1102 EMIF06-mSD02C3, U801 MCIMX7D7DVM10SC

Commit message: Created netlist with current components Foreward Annotation to Board
Parts:
- C1101, C1102, C1103, C1104, C1106: footprint (none) -> Capacitors_SMD:C_0402
- C1105: footprint (none) -> Capacitors_SMD:C_0603
- U801: footprint (none) -> NokiaRetroFit:BGA_541_075_19x19
Changed lines of the file:
@@
 F 0 "U801" H 3900 3000 60  0000 L CNN
 F 1 "MCIMX7D7DVM10SC" H 3900 2900 60  0000 L CNN
-F 2 "" H 1650 4700 60  0001 C CNN
+F 2 "NokiaRetroFit:BGA_541_075_19x19" H 1650 4700 60  0001 C CNN
 F 3 "" H 1650 4700 60  0001 C CNN
 	12   3900 3000
@@
 F 0 "J1101" H 11300 5400 60  0000 C CNN
 F 1 "MICRO_SD_HINGE" H 11250 5900 60  0000 C CNN
-F 2 "" V 11360 4850 60  0000 C CNN
+F 2 "" V 11360 4850 60  0001 C CNN
 F 3 "" V 11360 4850 60  0000 C CNN
 	1    11250 5350
@@
 $EndComp
 $Comp
-L GND #PWR0262
+L GND #PWR0261
 U 1 1 5944B647
 P 11200 6150
-F 0 "#PWR0262" H 11200 5900 50  0001 C CNN
+F 0 "#PWR0261" H 11200 5900 50  0001 C CNN
 F 1 "GND" H 11200 6000 50  0000 C CNN
 F 2 "" H 11200 6150 50  0000 C CNN
@@
 $EndComp
 $Comp
-L NVCC_3V3 #PWR0263
+L NVCC_3V3 #PWR0262
 U 1 1 5944C8E9
 P 10300 4450
-F 0 "#PWR0263" H 10300 4300 50  0001 C CNN
+F 0 "#PWR0262" H 10300 4300 50  0001 C CNN
 F 1 "NVCC_3V3" H 10300 4600 50  0000 C CNN
 F 2 "" H 10300 4450 50  0001 C CNN
@@
 F 0 "C1106" H 10675 8150 50  0000 L CNN
 F 1 "C" H 10675 7950 50  0000 L CNN
-F 2 "" H 10688 7900 50  0000 C CNN
+F 2 "Capacitors_SMD:C_0402" H 10688 7900 50  0001 C CNN
 F 3 "" H 10650 8050 50  0000 C CNN
 	1    10650 8050
@@
 	10650 7850 9950 7850
 $Comp
-L GND #PWR0264
+L GND #PWR0263
 U 1 1 5944DCC6
 P 10650 8250
-F 0 "#PWR0264" H 10650 8000 50  0001 C CNN
+F 0 "#PWR0263" H 10650 8000 50  0001 C CNN
 F 1 "GND" H 10650 8100 50  0000 C CNN
 F 2 "" H 10650 8250 50  0000 C CNN
@@
 	10650 8250 10650 8200
 $Comp
-L MEM_3V3 #PWR0265
+L MEM_3V3 #PWR0264
 U 1 1 5944DD41
 P 10300 8100
-F 0 "#PWR0265" H 10300 7950 50  0001 C CNN
+F 0 "#PWR0264" H 10300 7950 50  0001 C CNN
 F 1 "MEM_3V3" H 10300 8250 50  0000 C CNN
 F 2 "" H 10300 8100 50  0001 C CNN
@@
 Connection ~ 10000 8950
 $Comp
-L NVCC_SD3 #PWR0266
+L NVCC_SD3 #PWR0265
 U 1 1 5944E338
 P 10300 8650
-F 0 "#PWR0266" H 10300 8500 50  0001 C CNN
+F 0 "#PWR0265" H 10300 8500 50  0001 C CNN
 F 1 "NVCC_SD3" H 10300 8800 50  0000 C CNN
 F 2 "" H 10300 8650 50  0001 C CNN
@@
 	9950 10250 10000 10250
 $Comp
-L GND #PWR0267
+L GND #PWR0266
 U 1 1 5944E514
 P 10000 10400
-F 0 "#PWR0267" H 10000 10150 50  0001 C CNN
+F 0 "#PWR0266" H 10000 10150 50  0001 C CNN
 F 1 "GND" H 10000 10250 50  0000 C CNN
 F 2 "" H 10000 10400 50  0000 C CNN
@@
 F 0 "C1101" H 2725 3650 50  0000 L CNN
 F 1 "220n" H 2725 3450 50  0000 L CNN
-F 2 "" H 2738 3400 50  0000 C CNN
+F 2 "Capacitors_SMD:C_0402" H 2738 3400 50  0001 C CNN
 F 3 "" H 2700 3550 50  0000 C CNN
 	1    2700 3550
@@
 	2700 3200 2700 3400
 $Comp
-L NVCC_3V3 #PWR0268
+L NVCC_3V3 #PWR0267
 U 1 1 5944EF86
 P 2700 3200
-F 0 "#PWR0268" H 2700 3050 50  0001 C CNN
+F 0 "#PWR0267" H 2700 3050 50  0001 C CNN
 F 1 "NVCC_3V3" H 2700 3350 50  0000 C CNN
 F 2 "" H 2700 3200 50  0001 C CNN
@@
 Connection ~ 2700 3250
 $Comp
-L GND #PWR0269
+L GND #PWR0268
 U 1 1 5944F032
 P 2700 3750
-F 0 "#PWR0269" H 2700 3500 50  0001 C CNN
+F 0 "#PWR0268" H 2700 3500 50  0001 C CNN
 F 1 "GND" H 2700 3600 50  0000 C CNN
 F 2 "" H 2700 3750 50  0000 C CNN
@@
 F 0 "C1103" H 2725 6500 50  0000 L CNN
 F 1 "220n" H 2725 6300 50  0000 L CNN
-F 2 "" H 2738 6250 50  0000 C CNN
+F 2 "Capacitors_SMD:C_0402" H 2738 6250 50  0001 C CNN
 F 3 "" H 2700 6400 50  0000 C CNN
 	1    2700 6400
@@
 	2700 6150 2700 6250
 $Comp
-L GND #PWR0270
+L GND #PWR0269
 U 1 1 5944F9FC
 P 2700 6600
-F 0 "#PWR0270" H 2700 6350 50  0001 C CNN
+F 0 "#PWR0269" H 2700 6350 50  0001 C CNN
 F 1 "GND" H 2700 6450 50  0000 C CNN
 F 2 "" H 2700 6600 50  0000 C CNN
@@
 F 0 "C1102" H 2725 5300 50  0000 L CNN
 F 1 "220n" H 2725 5100 50  0000 L CNN
-F 2 "" H 2738 5050 50  0000 C CNN
+F 2 "Capacitors_SMD:C_0402" H 2738 5050 50  0001 C CNN
 F 3 "" H 2700 5200 50  0000 C CNN
 	1    2700 5200
@@
 	2700 4850 2700 5050
 $Comp
-L GND #PWR0271
+L GND #PWR0270
 U 1 1 5944FABA
 P 2700 5400
-F 0 "#PWR0271" H 2700 5150 50  0001 C CNN
+F 0 "#PWR0270" H 2700 5150 50  0001 C CNN
 F 1 "GND" H 2700 5250 50  0000 C CNN
 F 2 "" H 2700 5400 50  0000 C CNN
@@
 F 0 "C1104" H 2725 7700 50  0000 L CNN
 F 1 "220n" H 2725 7500 50  0000 L CNN
-F 2 "" H 2738 7450 50  0000 C CNN
+F 2 "Capacitors_SMD:C_0402" H 2738 7450 50  0001 C CNN
 F 3 "" H 2700 7600 50  0000 C CNN
 	1    2700 7600
@@
 	2700 7250 2700 7450
 $Comp
-L GND #PWR0272
+L GND #PWR0271
 U 1 1 5944FB14
 P 2700 7800
-F 0 "#PWR0272" H 2700 7550 50  0001 C CNN
+F 0 "#PWR0271" H 2700 7550 50  0001 C CNN
 F 1 "GND" H 2700 7650 50  0000 C CNN
 F 2 "" H 2700 7800 50  0000 C CNN
@@
 F 0 "C1105" H 2725 8700 50  0000 L CNN
 F 1 "2u2" H 2725 8500 50  0000 L CNN
-F 2 "" H 2738 8450 50  0000 C CNN
+F 2 "Capacitors_SMD:C_0603" H 2738 8450 50  0001 C CNN
 F 3 "" H 2700 8600 50  0000 C CNN
 	1    2700 8600
@@
 	2700 8350 2700 8450
 $Comp
-L GND #PWR0273
+L GND #PWR0272
 U 1 1 5944FC97
 P 2700 8800
-F 0 "#PWR0273" H 2700 8550 50  0001 C CNN
+F 0 "#PWR0272" H 2700 8550 50  0001 C CNN
 F 1 "GND" H 2700 8650 50  0000 C CNN
 F 2 "" H 2700 8800 50  0000 C CNN
@@
 Connection ~ 2700 4950
 $Comp
-L NVCC_SD1 #PWR0274
+L NVCC_SD1 #PWR0273
 U 1 1 594500AD
 P 2700 4850
-F 0 "#PWR0274" H 2700 4700 50  0001 C CNN
+F 0 "#PWR0273" H 2700 4700 50  0001 C CNN
 F 1 "NVCC_SD1" H 2700 5000 50  0000 C CNN
 F 2 "" H 2700 4850 50  0001 C CNN
@@
 	7050 9150 8350 9150
 $Comp
-L NVCC_1V8 #PWR0275
+L NVCC_1V8 #PWR0274
 U 1 1 595BDAEA
 P 2700 7250
-F 0 "#PWR0275" H 2700 7100 50  0001 C CNN
+F 0 "#PWR0274" H 2700 7100 50  0001 C CNN
 F 1 "NVCC_1V8" H 2700 7400 50  0000 C CNN
 F 2 "" H 2700 7250 50  0001 C CNN
