File: STORAGE.sch (KiCad schematic (older format))
At the start: 10 parts, among them J1101 MICRO_SD_HINGE, U1101 MTFC8GACAEAM-1M_WT, U1102 EMIF06-mSD02C3, U801 MCIMX7D7DVM10SC

Commit message: This branch moves from i.mx7 to STM32F4 CPU to be finished for Hackaday Prize 2017
Parts:
- removed C1101, C1102, C1103, C1104: 220n, Capacitors_SMD:C_0402, symbol C
- removed C1105: 2u2, Capacitors_SMD:C_0603, symbol C
- removed C1106: C, Capacitors_SMD:C_0402, symbol C
- removed U1101: MTFC8GACAEAM-1M_WT, symbol MTFC8GACAEAM-1M_WT
- removed U801: MCIMX7D7DVM10SC, NokiaRetroFit:BGA_541_075_19x19, symbol MCIMX7D7DVM10SC
Connections:
- net labels added: SD_CLK, SD_CMD, SD_D0, SD_D1, SD_D2, SD_D3
- net labels removed: CCM_CLKO2_32k, MEM_3V3, NVCC_1V8, NVCC_SD1, NVCC_SD2, NVCC_SD3, SAI1[0..6], SAI1_0, SAI1_1, SAI1_2, SAI1_3, SAI1_4, SAI1_5, SAI1_6, SAI2[0..3], SAI2_0, SAI2_1, SAI2_2, SAI2_3, SD1_CLK, SD1_CMD, SD1_D0, SD1_D1, SD1_D2, SD1_D3, SD1_WP, SD1_~CD, SD1_~RST, SD2_BUS0, SD2_BUS1, SD2_BUS2, SD2_BUS3, SD2_BUS4, SD2_BUS5, SD2_BUS6, SD2_BUS7, SD2_BUS8, SD2_BUS[0..8], SD2_CLK, SD2_CMD, SD2_D0, SD2_D1, SD2_D2, SD2_D3, SD2_WP, SD2_~CD, SD2_~RST, SD3_CLK, SD3_CMD, SD3_D0, SD3_D1, SD3_D2, SD3_D3, SD3_D4, SD3_D5, SD3_D6, SD3_D7
- wire segments 126 -> 34
Other:
- moved on the sheet: J1101

Commit message: Modification for STM32 adaption
For the Hackaday Prize 2017 I decided to switch to STM32 as CPU

*Power system was modified to just contain the charge IC,
*Boost converter for high voltage peripherals
*Buck converter for 3V3 for CPU and switchable NVCC_3V3
   for peripherie

CPU signals are routed and pinmux is done in firmware folder.

SD-Card has 4bit Interface

WiFi module ESP8266 is connected via UART

Wolfson Ausio codec is connected via SAI

Two digital microphones for noise canceling

Rumble Motor driver

LCD is connected via it's own I2C interface
Parts:
- J1101: footprint (none) -> Connectors:microSD_Card_Receptacle_Wuerth_693072010801
Connections:
- wire segments 34 -> 26
Other:
- moved on the sheet: J1101
Changed lines of the file:
@@
 EESchema Schematic File Version 2
-LIBS:3210retro-rescue
 LIBS:a7
 LIBS:ft232rl
@@
 LIBS:contrib
 LIBS:valves
-LIBS:stm32
+LIBS:tps62742
+LIBS:WM8994ECS
 LIBS:3210retro-cache
 EELAYER 26 0
 EELAYER END
-$Descr A3 16535 11693
+$Descr A4 11693 8268
 encoding utf-8
 Sheet 9 10
 Title "Nokia 3210 Retrofit"
-Date "2017-06-15"
-Rev "2"
+Date "2017-09-07"
+Rev "3"
 Comp "www.kurzschluss-blog.de"
-Comment1 "Retrofitting board for Nokia 3210 mobile phone"
-Comment2 ""
+Comment1 "Retro fitting board for Nokia 3210 mobile phone"
+Comment2 "STM32 Version"
 Comment3 ""
 Comment4 ""
@@
 L MICRO_SD_HINGE J1101
 U 1 1 5944B602
-P 12700 3800
-F 0 "J1101" H 12750 3850 60  0000 C CNN
-F 1 "MICRO_SD_HINGE" H 12700 4350 60  0000 C CNN
-F 2 "" V 12810 3300 60  0001 C CNN
-F 3 "" V 12810 3300 60  0000 C CNN
-	1    12700 3800
+P 7300 3750
+F 0 "J1101" H 7350 3800 60  0000 C CNN
+F 1 "MICRO_SD_HINGE" H 7300 4300 60  0000 C CNN
+F 2 "Connectors:microSD_Card_Receptacle_Wuerth_693072010801" V 7410 3250 60  0001 C CNN
+F 3 "" V 7410 3250 60  0000 C CNN
+	1    7300 3750
 	1    0    0    -1
 $EndComp
@@
 L GND #PWR0261
 U 1 1 5944B647
-P 12650 4600
-F 0 "#PWR0261" H 12650 4350 50  0001 C CNN
-F 1 "GND" H 12650 4450 50  0000 C CNN
-F 2 "" H 12650 4600 50  0000 C CNN
-F 3 "" H 12650 4600 50  0000 C CNN
-	1    12650 4600
+P 7250 4550
+F 0 "#PWR0261" H 7250 4300 50  0001 C CNN
+F 1 "GND" H 7250 4400 50  0000 C CNN
+F 2 "" H 7250 4550 50  0000 C CNN
+F 3 "" H 7250 4550 50  0000 C CNN
+	1    7250 4550
 	1    0    0    -1
 $EndComp
 Wire Wire Line
-	12650 4500 12650 4550
+	7250 4450 7250 4550
 Wire Wire Line
-	12650 4550 12650 4600
+	5400 4500 7550 4500
 Wire Wire Line
-	10800 4550 10900 4550
+	7550 4500 7550 4450
+Connection ~ 7250 4500
 Wire Wire Line
-	10900 4550 11000 4550
+	7450 4450 7450 4500
+Connection ~ 7450 4500
 Wire Wire Line
-	11000 4550 11750 4550
+	7350 4450 7350 4500
+Connection ~ 7350 4500
 Wire Wire Line
-	11750 4550 12650 4550
+	6500 3850 6350 3850
 Wire Wire Line
-	12650 4550 12750 4550
+	6350 3850 6350 4500
 Wire Wire Line
-	12750 4550 12850 4550
+	4750 3950 4050 3950
 Wire Wire Line
-	12850 4550 12950 4550
+	4750 4050 4050 4050
 Wire Wire Line
-	12950 4550 12950 4500
-Connection ~ 12650 4550
+	4050 3350 4750 3350
 Wire Wire Line
-	12850 4500 12850 4550
-Connection ~ 12850 4550
+	4750 3450 4050 3450
 Wire Wire Line
-	12750 4500 12750 4550
-Connection ~ 12750 4550
+	4750 3550 4050 3550
 Wire Wire Line
-	11900 3900 11750 3900
+	4750 3750 4050 3750
 Wire Wire Line
-	11750 3900 11750 4550
+	6500 4050 6250 4050
 Wire Wire Line
-	10150 4000 9450 4000
+	6250 3950 6500 3950
 Wire Wire Line
-	10150 4100 9450 4100
+	6500 3750 6250 3750
 Wire Wire Line
-	9450 3400 10150 3400
+	6250 3550 6500 3550
 Wire Wire Line
-	10150 3500 9450 3500
+	6500 3450 6250 3450
 Wire Wire Line
-	10150 3600 9450 3600
-Wire Wire Line
-	10150 3800 9450 3800
-Wire Wire Line
-	11900 4100 11650 4100
-Wire Wire Line
-	11650 4000 11900 4000
-Wire Wire Line
-	11900 3800 11650 3800
-Wire Wire Line
-	11650 3600 11900 3600
-Wire Wire Line
-	11900 3500 11650 3500
-Wire Wire Line
-	11650 3400 11900 3400
+	6250 3350 6500 3350
 $Comp
 L EMIF06-mSD02C3 U1102
 U 1 1 5944C05B
-P 10900 3700
-F 0 "U1102" H 11350 4150 60  0000 C CNN
-F 1 "EMIF06-mSD02C3" H 10900 3700 60  0000 C CNN
-F 2 "" H 11350 4150 60  0001 C CNN
-F 3 "" H 11350 4150 60  0001 C CNN
-	1    10900 3700
+P 5500 3650
+F 0 "U1102" H 5950 4100 60  0000 C CNN
+F 1 "EMIF06-mSD02C3" H 5500 3650 60  0000 C CNN
+F 2 "" H 5950 4100 60  0001 C CNN
+F 3 "" H 5950 4100 60  0001 C CNN
+	1    5500 3650
 	1    0    0    -1
 $EndComp
@@
 L NVCC_3V3 #PWR0262
 U 1 1 5944C8E9
-P 11750 2900
-F 0 "#PWR0262" H 11750 2750 50  0001 C CNN
-F 1 "NVCC_3V3" H 11750 3050 50  0000 C CNN
-F 2 "" H 11750 2900 50  0001 C CNN
-F 3 "" H 11750 2900 50  0001 C CNN
-	1    11750 2900
+P 6350 2850
+F 0 "#PWR0262" H 6350 2700 50  0001 C CNN
+F 1 "NVCC_3V3" H 6350 3000 50  0000 C CNN
+F 2 "" H 6350 2850 50  0001 C CNN
+F 3 "" H 6350 2850 50  0001 C CNN
+	1    6350 2850
 	1    0    0    -1
 $EndComp
 Wire Wire Line
-	11750 3700 11900 3700
+	6350 3650 6500 3650
 Wire Wire Line
-	11750 2900 11750 3000
+	6350 2850 6350 3650
 Wire Wire Line
-	11750 3000 11750 3700
+	6350 2950 5500 2950
 Wire Wire Line
-	11750 3000 10900 3000
+	5500 2950 5500 3050
+Connection ~ 6350 2950
 Wire Wire Line
-	10900 3000 10900 3100
-Connection ~ 11750 3000
+	5400 4350 5400 4500
+Connection ~ 6350 4500
 Wire Wire Line
-	10800 4400 10800 4550
-Connection ~ 11750 4550
+	5500 4350 5500 4500
+Connection ~ 5500 4500
 Wire Wire Line
-	10900 4400 10900 4550
-Connection ~ 10900 4550
-Wire Wire Line
-	11000 4400 11000 4550
-Connection ~ 11000 4550
-Text HLabel 9450 3400 0    60   BiDi ~ 0
+	5600 4350 5600 4500
+Connection ~ 5600 4500
+Text HLabel 4050 3350 0    60   BiDi ~ 0
 SD_D2
-Text HLabel 9450 3500 0    60   BiDi ~ 0
+Text HLabel 4050 3450 0    60   BiDi ~ 0
 SD_D3
-Text HLabel 9450 4000 0    60   BiDi ~ 0
+Text HLabel 4050 3950 0    60   BiDi ~ 0
 SD_D0
-Text HLabel 9450 4100 0    60   BiDi ~ 0
+Text HLabel 4050 4050 0    60   BiDi ~ 0
 SD_D1
-Text HLabel 9450 3800 0    60   Input ~ 0
+Text HLabel 4050 3750 0    60   Input ~ 0
 SD_CLK
-Text HLabel 9450 3600 0    60   Input ~ 0
+Text HLabel 4050 3550 0    60   Input ~ 0
 SD_CMD
 $EndSCHEMATC

Commit message: Placed a lot of components and routed the audio codec
The BGA of tha audio chipset is to small for regualr technology.
We do not use all of the pins of the chip so we ignore the other
pads and escape throug the balls of the other pad.
Parts:
- U1102: footprint (none) -> NokiaRetroFit:EMIF06-mSD02C3
Changed lines of the file:
@@
 LIBS:contrib
 LIBS:valves
-LIBS:tps62742
-LIBS:WM8994ECS
+LIBS:stm32
 LIBS:3210retro-cache
 EELAYER 26 0
@@
 F 0 "U1102" H 5950 4100 60  0000 C CNN
 F 1 "EMIF06-mSD02C3" H 5500 3650 60  0000 C CNN
-F 2 "" H 5950 4100 60  0001 C CNN
+F 2 "NokiaRetroFit:EMIF06-mSD02C3" H 5950 4100 60  0001 C CNN
 F 3 "" H 5950 4100 60  0001 C CNN
 	1    5500 3650

Commit message: Revision 1 of Layout
6layer board
through-hole via only (0.5/0.3mm drill)
0.2mm track width

https://hackaday.io/project/21263-nokia-3210-retro-fit-board/log/66914-prototype-pcb-done-there-comes-the-review
Parts:
- removed U1102: EMIF06-mSD02C3, NokiaRetroFit:EMIF06-mSD02C3, symbol EMIF06-mSD02C3
Connections:
- wire segments 26 -> 15
Changed lines of the file:
@@
 	7250 4450 7250 4550
-Wire Wire Line
-	5400 4500 7550 4500
 Wire Wire Line
 	7550 4500 7550 4450
@@
 	6350 3850 6350 4500
 Wire Wire Line
-	4750 3950 4050 3950
+	5550 3950 6500 3950
 Wire Wire Line
-	4750 4050 4050 4050
+	5550 4050 6500 4050
 Wire Wire Line
-	4050 3350 4750 3350
+	5550 3350 6500 3350
 Wire Wire Line
-	4750 3450 4050 3450
+	5550 3450 6500 3450
 Wire Wire Line
-	4750 3550 4050 3550
+	5550 3550 6500 3550
 Wire Wire Line
-	4750 3750 4050 3750
-Wire Wire Line
-	6500 4050 6250 4050
-Wire Wire Line
-	6250 3950 6500 3950
-Wire Wire Line
-	6500 3750 6250 3750
-Wire Wire Line
-	6250 3550 6500 3550
-Wire Wire Line
-	6500 3450 6250 3450
-Wire Wire Line
-	6250 3350 6500 3350
-$Comp
-L EMIF06-mSD02C3 U1102
-U 1 1 5944C05B
-P 5500 3650
-F 0 "U1102" H 5950 4100 60  0000 C CNN
-F 1 "EMIF06-mSD02C3" H 5500 3650 60  0000 C CNN
-F 2 "NokiaRetroFit:EMIF06-mSD02C3" H 5950 4100 60  0001 C CNN
-F 3 "" H 5950 4100 60  0001 C CNN
-	1    5500 3650
-	1    0    0    -1
-$EndComp
+	5550 3750 6500 3750
 $Comp
 L NVCC_3V3 #PWR0262
@@
 Wire Wire Line
 	6350 2850 6350 3650
+Text HLabel 5550 3350 0    60   BiDi ~ 0
+SD_D2
+Text HLabel 5550 3450 0    60   BiDi ~ 0
+SD_D3
+Text HLabel 5550 3950 0    60   BiDi ~ 0
+SD_D0
+Text HLabel 5550 4050 0    60   BiDi ~ 0
+SD_D1
+Text HLabel 5550 3750 0    60   Input ~ 0
+SD_CLK
+Text HLabel 5550 3550 0    60   Input ~ 0
+SD_CMD
 Wire Wire Line
-	6350 2950 5500 2950
-Wire Wire Line
-	5500 2950 5500 3050
-Connection ~ 6350 2950
-Wire Wire Line
-	5400 4350 5400 4500
-Connection ~ 6350 4500
-Wire Wire Line
-	5500 4350 5500 4500
-Connection ~ 5500 4500
-Wire Wire Line
-	5600 4350 5600 4500
-Connection ~ 5600 4500
-Text HLabel 4050 3350 0    60   BiDi ~ 0
-SD_D2
-Text HLabel 4050 3450 0    60   BiDi ~ 0
-SD_D3
-Text HLabel 4050 3950 0    60   BiDi ~ 0
-SD_D0
-Text HLabel 4050 4050 0    60   BiDi ~ 0
-SD_D1
-Text HLabel 4050 3750 0    60   Input ~ 0
-SD_CLK
-Text HLabel 4050 3550 0    60   Input ~ 0
-SD_CMD
+	6350 4500 7550 4500
 $EndSCHEMATC
