File: 3210retro.kicad_pcb (KiCad board)
At the start: 8 copper layers, 44 x 118 mm, 493 parts, among them J1001 TEST_1P, J901 GND, J902 GND, J903 GND, J904 GND, J905 GND, J906 GND, J907 GND, J908 GND, J909 GND, J910 GND, J911 GND, J912 GND, J913 GND, J914 GND, J915 GND, J916 GND, J917 GND, J918 GND, J919 GND, J920 GND, J921 GND, J922 GND, J923 GND, J924 GND, P101 USB_OTG, P102 NIMH, P103 LIPO, P104 DC, P105 EAR, P106 SPEAKER, P107 HEADPHONE, P108 RUMBLE, P109 RUMBLE, P301 SEPS525, P601 ESP_DBG, P602 BT_DBG, P603 WL_DBG, P604 WL_RS232, P801 JTAG, P802 A7, P803 M4, Q201 PZTA42, Q202 PZTA42, Q203 BCP51, Q501 MMBF170, Q701 MMBF170, SW701 SW_PUSH, SW702 C, SW703 1, SW704 4ghi, SW705 7pqrs, SW706 -, SW707 2abc, SW708 5jkl, SW709 8tuv, SW710 UP, SW711 3def, SW712 6mno, SW713 9wxyz, SW714 *+, SW715 DOWN, SW716 0space, SW717 #up, U1001 PF3000, U1301 LSM9DS1, U201 MAX1555, U202 BQ24400, U301 TPS61041DBV, U401 TS5A22366, U402 DRV8601, U403 WM8960CGEFL/V, U404 MP34DT01TR, U405 MP34DT01TR, U504 A7, U505 SIM_SLOT, U601 ESP-12E, U602 U.FL, U603 U.FL, U801 MCIMX7D7DVM10SC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

Commit message: This branch moves from i.mx7 to STM32F4 CPU to be finished for Hackaday Prize 2017
Parts:
- removed R901, R902: 0R, Resistors_SMD:R_0402
- moved C916 55.2 mm to (41.5, 92.8)
- moved C914 55.1 mm to (41.7, 91.3)
- moved C917 54.1 mm to (42.5, 99.5)
- moved R908 51.9 mm to (43.1, 90.0)
- moved C920 49.4 mm to (38.2, 97.3)
- moved C924 49.4 mm to (38.2, 94.6)
- moved C918 49.3 mm to (38.3, 96.1)
- moved C909 49.2 mm to (39.0, 91.6)
- moved C919 48.8 mm to (38.8, 85.0)
- moved C912 48.3 mm to (39.3, 88.7)
- moved C922 48.3 mm to (39.3, 89.9)
- moved C923 48.3 mm to (39.4, 83.8)
- moved C911 48.3 mm to (39.3, 86.6)
- moved C913 44.3 mm to (52.5, 83.0)
- moved C921 44.2 mm to (52.5, 82.0)
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Connections:
- C1018 pad 2: (no net) -> Net-(C1018-Pad2)
- C1106 pad 1: (no net) -> Net-(C1106-Pad1)
- C1308 pad 1: (no net) -> Net-(C1308-Pad1)
- C1309 pad 1: (no net) -> Net-(C1309-Pad1)
- C402 pad 1: (no net) -> Net-(C402-Pad1)
- C410 pad 1: (no net) -> Net-(C410-Pad1)
- C414 pad 1: (no net) -> Net-(C414-Pad1)
- C415 pad 1: (no net) -> Net-(C415-Pad1)
- C419 pad 2: (no net) -> /Audio Amplifier/MIC_IN
- FB402 pad 1: (no net) -> +3V3
- FB402 pad 2: (no net) -> Net-(FB402-Pad2)
- L401 pad 1: (no net) -> Net-(L401-Pad1)
- L402 pad 1: (no net) -> Net-(L402-Pad1)
- L403 pad 1: (no net) -> Net-(L403-Pad1)
- L404 pad 1: (no net) -> Net-(L404-Pad1)
- P108 pad 1: (no net) -> /Audio Amplifier/RMBL-
- P301 pad 1: (no net) -> Net-(P301-Pad1)
- P301 pad 35: (no net) -> Net-(P301-Pad35)
- P602 pad 2: (no net) -> Net-(P602-Pad2)
- P603 pad 2: (no net) -> Net-(P603-Pad2)
- P604 pad 2: (no net) -> Net-(P604-Pad2)
- P604 pad 3: (no net) -> Net-(P604-Pad3)
- P801 pad 7: (no net) -> Net-(P801-Pad7)
- R305 pad 2: (no net) -> Net-(R305-Pad2)
- R310 pad 2: (no net) -> /Display/DISPLAY_DATA9
- R311 pad 2: (no net) -> /Display/DISPLAY_DATA8
- R312 pad 2: (no net) -> /Display/DISPLAY_DATA7
- R313 pad 2: (no net) -> /Display/DISPLAY_DATA6
- R314 pad 2: (no net) -> /Display/DISPLAY_DATA5
- R315 pad 2: (no net) -> /Display/DISPLAY_DATA4
- R316 pad 2: (no net) -> /Display/DISPLAY_DATA3
- R317 pad 2: (no net) -> /Display/DISPLAY_DATA2
- R318 pad 2: (no net) -> /Display/DISPLAY_DATA1
- R319 pad 2: (no net) -> /Display/DISPLAY_DATA0
- R320 pad 2: (no net) -> /Display/DISPLAY_DATA10
- R321 pad 2: (no net) -> /Display/DISPLAY_DATA11
- R322 pad 2: (no net) -> /Display/DISPLAY_DATA12
- R611 pad 1: (no net) -> Net-(R611-Pad1)
- R612 pad 1: (no net) -> Net-(R612-Pad1)
- R613 pad 1: (no net) -> Net-(R613-Pad1)
- R614 pad 1: (no net) -> Net-(R614-Pad1)
- R615 pad 1: (no net) -> Net-(R615-Pad1)
- R616 pad 1: (no net) -> Net-(R616-Pad1)
- R617 pad 1: (no net) -> Net-(R617-Pad1)
- TP301 pad 1: (no net) -> Net-(TP301-Pad1)
- TP302 pad 1: (no net) -> Net-(TP302-Pad1)
- TP702 pad 1: (no net) -> Net-(TP702-Pad1)
- TP703 pad 1: (no net) -> Net-(TP703-Pad1)
- TP704 pad 1: (no net) -> Net-(TP704-Pad1)
- TP705 pad 1: (no net) -> Net-(TP705-Pad1)
- TP706 pad 1: (no net) -> Net-(TP706-Pad1)
- TP707 pad 1: (no net) -> Net-(TP707-Pad1)
- TP708 pad 1: (no net) -> Net-(TP708-Pad1)
- TP709 pad 1: (no net) -> Net-(TP709-Pad1)
- U202 pad 5: (no net) -> Net-(U202-Pad5)
- U401 pad A2: (no net) -> Net-(U401-PadA2)
- U401 pad B2: (no net) -> Net-(U401-PadB2)
- U401 pad C1: (no net) -> Net-(U401-PadC1)
- U401 pad C2: (no net) -> Net-(U401-PadC2)
- U401 pad C3: (no net) -> Net-(U401-PadC3)
- U401 pad D1: (no net) -> Net-(U401-PadD1)
- U401 pad D2: (no net) -> Net-(U401-PadD2)
- U401 pad D3: (no net) -> Net-(U401-PadD3)
- U504 pad 17: (no net) -> Net-(U504-Pad17)
- U504 pad 21: (no net) -> /Radio Module, GPS and SIM/HP_M
- U504 pad 23: (no net) -> /Radio Module, GPS and SIM/HP_L
- U504 pad 24: (no net) -> /Radio Module, GPS and SIM/HP_R
- U504 pad 26: (no net) -> /Audio Amplifier/SPK_+
- U504 pad 27: (no net) -> /Audio Amplifier/SPK_-
- U504 pad 3: (no net) -> Net-(U504-Pad3)
- U504 pad 38: (no net) -> Net-(U504-Pad38)
- U504 pad 4: (no net) -> Net-(U504-Pad4)
- U504 pad 5: (no net) -> Net-(U504-Pad5)
- U504 pad 6: (no net) -> Net-(U504-Pad6)
- U504 pad 7: (no net) -> Net-(U504-Pad7)
- U601 pad 11: (no net) -> Net-(U601-Pad11)
- U601 pad 12: (no net) -> Net-(U601-Pad12)
- U601 pad 13: (no net) -> Net-(U601-Pad13)
- U601 pad 14: (no net) -> Net-(U601-Pad14)
- U601 pad 2: (no net) -> Net-(U601-Pad2)
- U601 pad 4: (no net) -> Net-(U601-Pad4)
- U601 pad 5: (no net) -> Net-(U601-Pad5)
- U601 pad 6: (no net) -> Net-(U601-Pad6)
- U601 pad 7: (no net) -> Net-(U601-Pad7)
- U801 pad A02: (no net) -> /Controller/Mass storage/SD3_D1
- U801 pad A04: (no net) -> /Controller/Mass storage/SD1_D2
- U801 pad A05: (no net) -> /Controller/Mass storage/SD1_D0
- U801 pad A10: (no net) -> Net-(U801-PadA10)
- U801 pad A11: (no net) -> Net-(U801-PadA11)
- U801 pad A12: (no net) -> Net-(U801-PadA12)
- U801 pad A22: (no net) -> /Controller/LCD_DATA01
- U801 pad A23: (no net) -> /Controller/LCD_DATA03
- U801 pad A24: (no net) -> /Controller/LCD_DATA06
- U801 pad AA03: (no net) -> Net-(U801-PadAA03)
- U801 pad AA04: (no net) -> Net-(U801-PadAA04)
- U801 pad AA05: (no net) -> Net-(U801-PadAA05)
- U801 pad AA07: (no net) -> Net-(U801-PadAA07)
- U801 pad AA14: (no net) -> /Controller/DDR3 RAM /ODT1
- U801 pad AA22: (no net) -> /Controller/DDR3 RAM /CS1
- U801 pad AB01: (no net) -> Net-(U801-PadAB01)
- U801 pad AB02: (no net) -> Net-(U801-PadAB02)
- U801 pad AB06: (no net) -> Net-(U801-PadAB06)
- U801 pad AB20: (no net) -> /Controller/DDR3 RAM /DRAM_ADDR15
- U801 pad AC01: (no net) -> Net-(U801-PadAC01)
- U801 pad AC02: (no net) -> Net-(U801-PadAC02)
- U801 pad AD24: Net-(R901-Pad2) -> /Controller/DDR3 RAM /SDCLK0_P
- U801 pad AD25: Net-(R902-Pad2) -> /Controller/DDR3 RAM /SDCLK0_N
- U801 pad AE03: (no net) -> Net-(U801-PadAE03)
- U801 pad B01: (no net) -> /Controller/Mass storage/SD3_D7
- U801 pad B02: (no net) -> /Controller/Mass storage/SD3_D0
- U801 pad B04: (no net) -> /Controller/Mass storage/SD1_~RST
- U801 pad B05: (no net) -> /Controller/Mass storage/SD1_CLK
- U801 pad B10: (no net) -> Net-(U801-PadB10)
- U801 pad B11: (no net) -> Net-(U801-PadB11)
- U801 pad B12: (no net) -> Net-(U801-PadB12)
- U801 pad B22: (no net) -> /Controller/LCD_DATA02
- U801 pad B23: (no net) -> /Controller/LCD_DATA05
- U801 pad B24: (no net) -> /Controller/LCD_DATA10
- U801 pad B25: (no net) -> /Controller/LCD_DATA16
- U801 pad C01: (no net) -> /Controller/Mass storage/SD3_CLK
- U801 pad C02: (no net) -> /Controller/Mass storage/SD3_D6
- U801 pad C04: (no net) -> CCM_CLKO2_32k
- U801 pad C05: (no net) -> /Controller/Mass storage/SD1_CMD
- U801 pad C06: (no net) -> /Controller/Mass storage/SD1_~CD
- U801 pad C07: (no net) -> Net-(U801-PadC07)
- U801 pad C10: (no net) -> Net-(U801-PadC10)
- U801 pad C11: (no net) -> /Controller/Mass storage/SAI1_5
- U801 pad C12: (no net) -> /Controller/Mass storage/SAI1_3
- U801 pad C22: (no net) -> /Controller/LCD_DATA04
- U801 pad C23: (no net) -> /Controller/LCD_DATA09
- U801 pad C24: (no net) -> /Controller/LCD_DATA15
- U801 pad C25: (no net) -> /Controller/LCD_DATA20
- U801 pad D05: (no net) -> /Controller/Mass storage/SD1_D3
- U801 pad D06: (no net) -> /Controller/Mass storage/SD1_D1
- U801 pad D08: (no net) -> /Controller/Mass storage/SAI2_2
- U801 pad D09: (no net) -> /Controller/Mass storage/SAI2_3
- U801 pad D11: (no net) -> /Controller/Mass storage/SAI1_6
- U801 pad D12: (no net) -> /Controller/Mass storage/SAI1_2
- U801 pad D21: (no net) -> /Controller/LCD_DATA00
- U801 pad D23: (no net) -> /Controller/LCD_DATA14
- U801 pad D24: (no net) -> /Controller/LCD_DATA19
- U801 pad D25: (no net) -> /Controller/LCD_DATA22
- U801 pad E01: (no net) -> /Controller/Mass storage/SD3_CMD
- U801 pad E02: (no net) -> /Controller/Mass storage/SD3_D5
- U801 pad E08: (no net) -> /Controller/Mass storage/SAI2_1
- U801 pad E09: (no net) -> /Controller/Mass storage/SAI2_0
- U801 pad E10: (no net) -> /Controller/Mass storage/SAI1_0
- U801 pad E11: (no net) -> /Controller/Mass storage/SAI1_4
- U801 pad E12: (no net) -> /Controller/Mass storage/SAI1_1
- U801 pad E21: (no net) -> /Controller/LCD_DATA08
- U801 pad E22: (no net) -> /Controller/LCD_DATA13
- U801 pad E23: (no net) -> /Controller/LCD_DATA18
- U801 pad E24: (no net) -> /Controller/LCD_DATA21
- U801 pad F01: (no net) -> /Controller/Mass storage/SD3_D3
- U801 pad F02: (no net) -> /Controller/Mass storage/SD3_D4
- U801 pad F20: (no net) -> /Controller/LCD_DATA07
- U801 pad F21: (no net) -> /Controller/LCD_DATA12
- U801 pad G01: (no net) -> Net-(U1101-PadK5)
- U801 pad G02: (no net) -> /Controller/Mass storage/SD3_D2
- U801 pad G05: (no net) -> /Controller/AT_UART0
- U801 pad G06: (no net) -> Net-(U801-PadG06)
- U801 pad G20: (no net) -> /Controller/LCD_DATA11
- U801 pad G21: (no net) -> /Controller/LCD_DATA17
- U801 pad G23: (no net) -> /Controller/LCD_DATA23
- U801 pad G25: (no net) -> /Audio Amplifier/RMBL_EN
- U801 pad H03: (no net) -> /Controller/AT_UART1
- U801 pad H04: (no net) -> /Controller/AT_UART3
- U801 pad H05: (no net) -> /Controller/AT_UART2
- U801 pad H06: (no net) -> Net-(U801-PadH06)
- U801 pad H20: (no net) -> Net-(U801-PadH20)
- U801 pad H21: (no net) -> Net-(U801-PadH21)
- U801 pad H24: (no net) -> Net-(U801-PadH24)
- U801 pad H25: (no net) -> Net-(U801-PadH25)
- U801 pad J01: (no net) -> Net-(U1101-PadH5)
- U801 pad J05: (no net) -> Net-(U801-PadJ05)
- U801 pad J06: (no net) -> Net-(U801-PadJ06)
- U801 pad J20: (no net) -> Net-(U801-PadJ20)
- U801 pad J21: (no net) -> Net-(U801-PadJ21)
- U801 pad J24: (no net) -> Net-(U801-PadJ24)
- U801 pad J25: (no net) -> Net-(U801-PadJ25)
- U801 pad K02: (no net) -> /Controller/USB and 9-axis IMU/IMU_SCL
- U801 pad K03: (no net) -> /Controller/USB and 9-axis IMU/IMU_SDA
- U801 pad K05: (no net) -> Net-(U801-PadK05)
- U801 pad K06: (no net) -> Net-(U801-PadK06)
- U801 pad K20: (no net) -> Net-(U801-PadK20)
- U801 pad K21: (no net) -> Net-(U801-PadK21)
- U801 pad K23: (no net) -> Net-(U801-PadK23)
- U801 pad K24: (no net) -> Net-(U801-PadK24)
- U801 pad K25: (no net) -> /Controller/UART7_CTS
- U801 pad L01: (no net) -> Net-(U801-PadL01)
- U801 pad L02: (no net) -> Net-(U801-PadL02)
- U801 pad L20: (no net) -> /Controller/UART7_RTS
- U801 pad L21: (no net) -> /Controller/HST_DL1
- U801 pad L22: (no net) -> /Controller/HST_DL0
- U801 pad L23: (no net) -> /Controller/GPIO2_D11
- U801 pad L24: (no net) -> /Controller/GPIO2_D10
- U801 pad L25: (no net) -> /Controller/GPIO2_D9
- U801 pad M01: (no net) -> /Controller/BT2
- U801 pad M02: (no net) -> /Controller/BT3
- U801 pad M05: (no net) -> /Controller/BT1
- U801 pad M06: (no net) -> /Controller/BT0
- U801 pad M23: (no net) -> /Controller/GPIO2_D8
- U801 pad N01: (no net) -> /Controller/PWM4_OUT
- U801 pad N05: (no net) -> /Controller/PWM3_OUT
- U801 pad N06: (no net) -> Net-(U801-PadN06)
- U801 pad P01: (no net) -> Net-(U801-PadP01)
- U801 pad P03: (no net) -> Net-(U801-PadP03)
- U801 pad P06: (no net) -> Net-(U801-PadP06)
- U801 pad R05: (no net) -> /Controller/BT_EN
- U801 pad T01: (no net) -> /Controller/IMU_EN
- U801 pad T02: (no net) -> /Controller/IMU_DRDY_M
- U801 pad T03: (no net) -> /Controller/IMU_INT_M
- U801 pad T05: (no net) -> /Controller/IMU_INT2
- U801 pad T06: (no net) -> /Controller/IMU_INT1
- U801 pad V04: (no net) -> Net-(U801-PadV04)
- U801 pad Y01: (no net) -> Net-(U801-PadY01)
- U801 pad Y02: (no net) -> Net-(U801-PadY02)
- U801 pad Y03: (no net) -> Net-(U801-PadY03)
- U801 pad Y04: (no net) -> Net-(U801-PadY04)
- U801 pad Y05: (no net) -> Net-(U801-PadY05)
- U801 pad Y07: (no net) -> Net-(U801-PadY07)
- U801 pad Y08: (no net) -> Net-(U801-PadY08)
- U901 pad J1: (no net) -> Net-(U901-PadJ1)
- U901 pad J9: (no net) -> Net-(U901-PadJ9)
- U901 pad L1: (no net) -> Net-(U901-PadL1)
- U901 pad L9: (no net) -> Net-(U901-PadL9)
- U901 pad M7: (no net) -> Net-(U901-PadM7)
- U902 pad J1: (no net) -> Net-(U902-PadJ1)
- U902 pad J9: (no net) -> Net-(U902-PadJ9)
- U902 pad L1: (no net) -> Net-(U902-PadL1)
- U902 pad L9: (no net) -> Net-(U902-PadL9)
- U902 pad M7: (no net) -> Net-(U902-PadM7)
Routing:
- net /Controller/DDR3 RAM /SDCLK0_N: track 0.00 -> 60.0 mm, vias 0 -> 3
- net /Controller/DDR3 RAM /SDCLK0_P: track 0.00 -> 59.6 mm, vias 0 -> 1
- net /Controller/DDR3 RAM /DRAM_ADDR5: track 17.5 -> 0.00 mm
- net /Controller/DDR3 RAM /SDCKE1: track 0.00 -> 15.3 mm
- net /Controller/DDR3 RAM /DRAM_ADDR7: track 40.0 -> 55.2 mm, vias 2 -> 3
- net /Controller/DDR3 RAM /DRAM_DATA26: track 2.47 -> 16.9 mm
- net /Controller/DDR3 RAM /DRAM_DATA27: track 2.17 -> 15.9 mm
- net /Controller/DDR3 RAM /DRAM_DATA29: track 2.92 -> 15.3 mm
- net /Controller/DDR3 RAM /DQM3: track 2.98 -> 15.0 mm
- net /Controller/DDR3 RAM /DRAM_DATA24: track 1.78 -> 13.4 mm
- net /Controller/DDR3 RAM /DRAM_ADDR14: track 20.6 -> 10.7 mm
- net /Controller/DDR3 RAM /SDQS3_P: track 3.05 -> 12.9 mm
- net /Controller/DDR3 RAM /DRAM_ADDR6: track 22.3 -> 12.7 mm
- net /Controller/DDR3 RAM /DRAM_ADDR0: track 18.9 -> 10.1 mm
- net /Controller/DDR3 RAM /DRAM_ADDR3: track 17.3 -> 8.87 mm
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Other:
- net class DDR_external: clearance 0.1 -> 0.135; trace_width 0.125 -> 0.1
- net class Default: trace_width 0.15 -> 0.25

Commit message: Placed a lot of components and routed the audio codec
The BGA of tha audio chipset is to small for regualr technology.
We do not use all of the pins of the chip so we ignore the other
pads and escape throug the balls of the other pad.
Parts:
- removed BT1001: LI_BAT, Pin_Headers:Pin_Header_Straight_1x02
- removed C1001, C1002, C1004, C1022, C604: 1u, Capacitors_SMD:C_0603
- removed C1003, C1006, C1011, C1105, C1215, C1223, C1224, C1225, C1230, C1234, C1236, C1237, C1238, C1303, C1304, C818: 2u2, Capacitors_SMD:C_0603
- removed C1005, C1008, C1013, C1018, C1027, C1028, C1029, C1030, C1208: 4u7, Capacitors_SMD:C_0603
- removed C1007: 10uF, Capacitors_SMD:C_0603
- removed C1009, C1016, C1019: 100nF, Capacitors_SMD:C_0402
- removed C1010, C1012, C1015: 1uF, Capacitors_SMD:C_0603
- removed C1014: 220nF, Capacitors_SMD:C_0402
- removed C1017, C1020, C1021, C1023, C1024, C1025, C1026, C205, C217, C606, C907: 100n, Capacitors_SMD:C_0402
- removed C1031, C1034: 22uF, Capacitors_SMD:C_0603
- removed C1032, C1033, C1035, C1036, C1037, C1038, C1039, C1040, C1041, C1042, C1043, C1044, C1217, C1220, C1221, C906, C923, C924, C938, C939: 22u, Capacitors_SMD:C_0603
- removed C1101, C1102, C1103, C1104, C1201, C1202, C1203, C1204, C1205, C1206, C1207, C1209, C1210, C1211, C1212, C1213, C1214, C1216, C1218, C1219, C1222, C1226, C1227, C1228, C1229, C1231, C1232, C1233, C1235, C1301, C1302, C1305, C1306, C901, C902, C903, C904, C905, C908, C909, C910, C911, C912, C913, C914, C915, C916, C917, C918, C919, C920, C921, C922, C925, C926, C927, C928, C929, C930, C931, C932, C933, C934, C935, C936, C937, C940: 220n, Capacitors_SMD:C_0402
- removed C1106: C, Capacitors_SMD:C_0402
- removed C1307, C201, C218, C605: 10u, Capacitors_SMD:C_0603
- removed C208, C216, C421, C422: 1n, Capacitors_SMD:C_0402
- removed C211: 330n, Capacitors_SMD:C_0603
- removed C212: 2n2, Capacitors_SMD:C_0402
- removed C213: 47u, Capacitors_SMD:C_0805
- removed C214: 4p7, Capacitors_SMD:C_0402
- removed C602: 1p, Capacitors_SMD:C_0402
- removed C603: 2p4, Capacitors_SMD:C_0402
- removed C816, C817: 470n, Capacitors_SMD:C_0402
- removed D1001, D801: D_Schottky, Diodes_SMD:SOD-123
- removed D201: BZT52-C5V1, Diodes_SMD:SOD-123
- removed D202, D204, D206, D207: MMSD914LT, Diodes_SMD:SOD-123
- removed D203: S1A, Diodes_SMD:SOD-123
- removed D205: ZHCS1000, Diodes_SMD:SOD-123
- removed D401, D402, D403: D_TVS_ALT, Diodes_SMD:SOD-123
- removed FB401: FILTER, Choke_SMD:Choke_SMD_1206_Standard
- removed J1001: TEST_1P, NokiaRetroFit:TP
- removed J901, J902, J903, J904, J905, J906, J907, J908, J909, J910, J911, J912, J913, J914, J915, J916, J917, J918, J919, J920, J921, J922, J923, J924: GND, NokiaRetroFit:TP
- removed L1001, L1201, L301, L302, L801: 100R, Choke_SMD:Choke_SMD_1206_Standard
- removed L1002, L1003, L1004, L1005, L1006: 1u5H, Choke_SMD:Choke_SMD_1206_Standard
- removed L401, L402, L403, L404, L405, L406, L407: 120R@100MHz, Choke_SMD:Choke_SMD_1206_Standard
- removed L601: 1n3, Choke_SMD:Choke_SMD_1206_Standard
- removed L602: 2n2, Choke_SMD:Choke_SMD_1206_Standard
- removed L603: 0, Choke_SMD:Choke_SMD_1206_Standard
- removed L604: 1n8, Choke_SMD:Choke_SMD_1206_Standard
- removed P102: NIMH, Pin_Headers:Pin_Header_Straight_2x01
- removed P103: LIPO, Pin_Headers:Pin_Header_Straight_2x01
- removed P104: DC, Pin_Headers:Pin_Header_Straight_2x01
- removed P105: EAR, Pin_Headers:Pin_Header_Straight_2x01
- removed P106: SPEAKER, Pin_Headers:Pin_Header_Straight_2x01
- removed P108: RUMBLE, Pin_Headers:Pin_Header_Straight_1x02
- removed P601: ESP_DBG, Pin_Headers:Pin_Header_Straight_1x02
- removed P602: BT_DBG, Pin_Headers:Pin_Header_Straight_1x02
- removed P603: WL_DBG, Pin_Headers:Pin_Header_Straight_1x02
- removed P604: WL_RS232, Pin_Headers:Pin_Header_Straight_1x03
- removed P802: A7, Pin_Headers:Pin_Header_Straight_1x02
- removed P803: M4, Pin_Headers:Pin_Header_Straight_1x02
- removed Q201, Q202: PZTA42, TO_SOT_Packages_SMD:SOT-223
- removed Q203: BCP51, TO_SOT_Packages_SMD:SOT-223
- removed R1001, R1002: R, Resistors_SMD:R_0402
- removed R1003, R907, R909: 470R, Resistors_SMD:R_0402
- removed R1004: 100K, Resistors_SMD:R_0402
- removed R1005, R1006, R1007, R1008, R1009, R1201, R1202, R1203, R1204, R906: 0R, Resistors_SMD:R_0402
- removed R1301: 200R, Resistors_SMD:R_0402
- removed R216: 1M, Resistors_SMD:R_0402
- removed R315, R316, R317, R318, R319, R320, R321, R322: 100, Resistors_SMD:R_0402
- removed R406: 20k, Resistors_SMD:R_0402
- removed R407: 33k, Resistors_SMD:R_0402
- removed R602, R604, R605, R606, R607, R608, R609, R610, R611, R612, R613, R614, R615, R616, R617, R810, R814, R815: 0, Resistors_SMD:R_0402
- removed R603, R618: 100k, Resistors_SMD:R_0402
- removed R808, R904, R905: 10k, Resistors_SMD:R_0402
- removed R809: 4k7, Resistors_SMD:R_0402
- removed R811, R812: 1k, Resistors_SMD:R_0402
- removed R813: 47k, Resistors_SMD:R_0402
- removed R903, R908, R910: 240R, Resistors_SMD:R_0402
- removed TP1201, TP1202, TP1203, TP1204, TP1205, TP1206, TP1207, TP1208, TP302: TP, NokiaRetroFit:TP
- removed U1001: PF3000, Housings_DFN_QFN:QFN-48-1EP_7x7mm_Pitch0.5mm
- removed U602, U603: U.FL, NokiaRetroFit:Foil_Button
- removed U901, U902: MT41K256M16HA-125, NokiaRetroFit:FBGA_96_x16
- removed Y601: ANT1/BT, SMD_Packages:1Pin
- removed Y602: ANT2/WL, SMD_Packages:1Pin
- added C306: 100n, Capacitors_SMD:C_0402_NoSilk, F.Cu at (109.4, 72.6)
- added C307: 100n, Capacitors_SMD:C_0402_NoSilk, F.Cu at (109.4, 73.5)
- added J1101: MICRO_SD_HINGE, Connectors:microSD_Card_Receptacle_Wuerth_693072010801, B.Cu at (109.7, 105.6)
- added J801: TEST_2P, Wire_Pads:SolderWirePad_2x_1mmDrill, F.Cu at (226.4, 65.4)
- added TP101: TP, NokiaRetroFit:TP, F.Cu at (213.5, 76.3)
- added U1102: EMIF06-mSD02C3, NokiaRetroFit:EMIF06-mSD02C3, F.Cu at (110.7, 99.0)
- added U203: TPS61021A, Housings_SON:Texas_S-PVSON-N8_ThermalVias, B.Cu at (107.1, 140.4)
- added U501: SN74AVC2T244, NokiaRetroFit:SN74AVC2T244, B.Cu at (103.5, 98.8)
- added U502: SN74AVC2T244, NokiaRetroFit:SN74AVC2T244, B.Cu at (95.6, 75.2)
- added U503: SN74AVC2T244, NokiaRetroFit:SN74AVC2T244, B.Cu at (92.8, 71.9)
- added U506: SN74AVC2T244, NokiaRetroFit:SN74AVC2T244, B.Cu at (87.1, 84.3)
- added Y801: 32kHz, Crystals:Crystal_SMD_SeikoEpson_MC146-4pin_6.7x1.5mm_HandSoldering, B.Cu at (81.5, 124.7)
- added Y802: 24MHz, Crystals:Crystal_SMD_SeikoEpson_MC146-4pin_6.7x1.5mm_HandSoldering, B.Cu at (84.1, 124.7)
- C1308: footprint Capacitors_SMD:C_0603 -> Capacitors_SMD:C_0402_NoSilk
- C1309, C504, C505, C506, C507: footprint Capacitors_SMD:C_0402 -> Capacitors_SMD:C_0402_NoSilk
- C202, C203, C502, L201, L303, P801, U201, U505: moved to B.Cu
- C204, C206, C207, C209, C210, C215, C219, C301, C302, C304, C401, C402, C403, C407, C417, C418, C420, C501, C503, C601, C801, C802, C803, C804, C809: footprint Capacitors_SMD:C_0402 -> Capacitors_SMD:C_0402_NoSilk; moved to B.Cu
- C220, C303, C305, C404, C410, C412, C413: footprint Capacitors_SMD:C_0603 -> Capacitors_SMD:C_0402_NoSilk; moved to B.Cu
- C405: value 4u7 -> 10n; footprint Capacitors_SMD:C_0603 -> Capacitors_SMD:C_0402_NoSilk; moved to B.Cu
- C406: value 100n -> 1u; footprint Capacitors_SMD:C_0402 -> Capacitors_SMD:C_0402_NoSilk; moved to B.Cu
- C408: value 4u7 -> 100n; footprint Capacitors_SMD:C_0603 -> Capacitors_SMD:C_0402_NoSilk; moved to B.Cu
- C409: value 1u -> 100n; footprint Capacitors_SMD:C_0603 -> Capacitors_SMD:C_0402_NoSilk; moved to B.Cu
- C411, C419: value 1u -> 4u7; footprint Capacitors_SMD:C_0603 -> Capacitors_SMD:C_0402_NoSilk; moved to B.Cu
- C414, C415: value 100u -> 100n; footprint Capacitors_SMD:c_elec_3x5.3 -> Capacitors_SMD:C_0402_NoSilk; moved to B.Cu
- C416: value 100n -> 4u7; footprint Capacitors_SMD:C_0402 -> Capacitors_SMD:C_0402_NoSilk; moved to B.Cu
- C805, C810: value 220n -> 100n; footprint Capacitors_SMD:C_0402 -> Capacitors_SMD:C_0402_NoSilk; moved to B.Cu
- C806: value 22u -> 2u2; footprint Capacitors_SMD:C_0603 -> Capacitors_SMD:C_0402_NoSilk; moved to B.Cu
- C807: value 220n -> 2u2; footprint Capacitors_SMD:C_0402 -> Capacitors_SMD:C_0402_NoSilk; moved to B.Cu
- C808, C814: value 2u2 -> 100n; footprint Capacitors_SMD:C_0603 -> Capacitors_SMD:C_0402_NoSilk; moved to B.Cu
- C811, C812, C813: value 470n -> 100n; footprint Capacitors_SMD:C_0402 -> Capacitors_SMD:C_0402_NoSilk; moved to B.Cu
- C815: value 2u2 -> 1u; footprint Capacitors_SMD:C_0603 -> Capacitors_SMD:C_0402_NoSilk; moved to B.Cu
- D301: footprint Diodes_SMD:SOD-123 -> Diodes_SMD:D_0805; moved to B.Cu
- L202: value 47u -> 2u2; moved to B.Cu
- P107: footprint Pin_Headers:Pin_Header_Straight_1x05 -> NokiaRetroFit:PJ_320_D; moved to B.Cu
- R101, R304, R323, R501, R502, R503, R504, R505, R701, R702, R703, R704, R705, R706, R707, R708: footprint Resistors_SMD:R_0402 -> Resistors_SMD:R_0402_NoSilk
- R201, R202, R203, R204, R207, R208, R217, R218, R301, R302, R401, R402, R601, R801, R804, R805, R806, R807: footprint Resistors_SMD:R_0402 -> Resistors_SMD:R_0402_NoSilk; moved to B.Cu
- R205: value 1k -> 0; footprint Resistors_SMD:R_0402 -> Resistors_SMD:R_0402_NoSilk; moved to B.Cu
- R206: value 6k81 -> 0; footprint Resistors_SMD:R_0402 -> Resistors_SMD:R_0402_NoSilk; moved to B.Cu
- R209: value 0R05 -> 0; footprint Resistors_SMD:R_0402 -> Resistors_SMD:R_0402_NoSilk; moved to B.Cu
- R210: value 1k1 -> 0; footprint Resistors_SMD:R_0402 -> Resistors_SMD:R_0402_NoSilk; moved to B.Cu
- R211, R214: value 100k -> 0; footprint Resistors_SMD:R_0402 -> Resistors_SMD:R_0402_NoSilk; moved to B.Cu
- R212: value 120 -> 0; footprint Resistors_SMD:R_0402 -> Resistors_SMD:R_0402_NoSilk; moved to B.Cu
- R213: value 220 -> 0; footprint Resistors_SMD:R_0402 -> Resistors_SMD:R_0402_NoSilk; moved to B.Cu
- R215, R803: value 100k -> 10k; footprint Resistors_SMD:R_0402 -> Resistors_SMD:R_0402_NoSilk; moved to B.Cu
- R303: value 70k -> 68k; footprint Resistors_SMD:R_0402 -> Resistors_SMD:R_0402_NoSilk
- R305, R306, R307, R310, R311: value 100 -> 560; footprint Resistors_SMD:R_0402 -> Resistors_SMD:R_0402_NoSilk
- R308, R309, R312, R313, R314: value 100 -> 1k; footprint Resistors_SMD:R_0402 -> Resistors_SMD:R_0402_NoSilk
- R403, R802: value 0 -> 10k; footprint Resistors_SMD:R_0402 -> Resistors_SMD:R_0402_NoSilk; moved to B.Cu
- R404, R405: value 20k -> 20; footprint Resistors_SMD:R_0402 -> Resistors_SMD:R_0402_NoSilk; moved to B.Cu
- U1301: footprint NokiaRetroFit:LSM9DS1 -> Housings_LGA:LGA-24L_3x3.5mm_Pitch0.43mm
- U202: value BQ24400 -> TPS62742; footprint SMD_Packages:SOIC-8-N -> NokiaRetroFit:TPS6274x; moved to B.Cu
- U301: footprint TO_SOT_Packages_SMD:SOT-23 -> Housings_DFN_QFN:DFN-6-1EP_2x2mm_Pitch0.65mm; moved to B.Cu
- U401: value TS5A22366 -> LD3985G18R_TSOT23; footprint NokiaRetroFit:TS5A22366 -> TO_SOT_Packages_SMD:TSOT-23-5; moved to B.Cu
- U402: footprint NokiaRetroFit:DRV8601 -> Housings_DFN_QFN:DFN-8-1EP_3x3mm_Pitch0.65mm; moved to B.Cu
- U403: value WM8960CGEFL/V -> WM8994ECS/R; footprint buttons:DRV8601 -> NokiaRetroFit:WM8994ECS_SPECIAL; moved to B.Cu
- U801: value MCIMX7D7DVM10SC -> STM32F756VGTx; footprint NokiaRetroFit:BGA_541_075_19x19 -> Housings_QFP:TQFP-100-1EP_14x14mm_Pitch0.5mm
- moved R101 498.7 mm to (98.9, 155.9), turned to 90 degrees
- moved R807 473.9 mm to (69.2, 149.8), turned to 90 degrees
- moved P107 473.6 mm to (91.6, 157.1), turned to 90 degrees
- moved R805 467.6 mm to (70.2, 149.8), turned to 270 degrees
- moved R806 464.3 mm to (68.2, 149.8), turned to 90 degrees
- moved R804 453.1 mm to (71.2, 149.8), turned to 270 degrees
- moved R801 452.7 mm to (69.7, 147.9), turned to 180 degrees
- moved C803 452.1 mm to (84.1, 130.1)
- moved C804 451.2 mm to (84.1, 119.3)
- moved C802 448.9 mm to (81.5, 119.3)
- moved C507 446.7 mm to (83.9, 80.7), turned to 90 degrees
- moved R504 445.5 mm to (85.2, 81.3), turned to 180 degrees
- moved C801 445.3 mm to (81.5, 130.1)
- moved C506 442.7 mm to (92.4, 99.7)
- moved C502 441.6 mm to (85.2, 89.3)
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Connections:
- net /Display/DISPLAY_DATA8 renamed /Controller/I2C3_SDA
- net /Display/DISPLAY_DATA9 renamed /Controller/I2C3_SCL
- C301 pad 1: NVCC_1V8 -> 18V_BST
- C302 pad 1: NVCC_1V8 -> 18V_BST
- C401 pad 1: NVCC_3V3 -> GND
- C401 pad 2: Net-(C401-Pad2) -> NVCC_3V3
- C403 pad 1: NVCC_3V3 -> GND
- C403 pad 2: Net-(C401-Pad2) -> NVCC_3V3
- C404 pad 1: VDD_SPK -> GND
- C404 pad 2: GNDA -> NVCC_3V3
- C405 pad 1: VDD_SPK -> Net-(C405-Pad1)
- C405 pad 2: GNDA -> GND
- C406 pad 1: +3.3VDAC -> GND
- C406 pad 2: GNDA -> NVCC_3V3
- C408 pad 1: /Audio Amplifier/MIC_BIAS -> GND
- C408 pad 2: GNDA -> NVCC_1V8
- C409 pad 1: +3.3VDAC -> GND
- C409 pad 2: GNDA -> NVCC_1V8
- C410 pad 1: Net-(C410-Pad1) -> GND
- C410 pad 2: GNDA -> NVCC_1V8
- C411 pad 1: +3.3VDAC -> GND
- C411 pad 2: GNDA -> Net-(C411-Pad2)
- C412 pad 1: +3.3VDAC -> GND
- C412 pad 2: GNDA -> Net-(C412-Pad2)
- C413 pad 1: +3.3VDAC -> Net-(C413-Pad1)
- C413 pad 2: GNDA -> GND
- C414 pad 1: Net-(C414-Pad1) -> GND
- C415 pad 1: Net-(C415-Pad1) -> GND
- C416 pad 1: NVCC_3V3 -> GND
- C416 pad 2: GND -> Net-(C416-Pad2)
- C417 pad 1: NVCC_3V3 -> Net-(C417-Pad1)
- C417 pad 2: GND -> Net-(C417-Pad2)
- C418 pad 1: NVCC_3V3 -> Net-(C418-Pad1)
- C418 pad 2: GND -> /Audio Amplifier/HPL
- C419 pad 1: Net-(C419-Pad1) -> GND
- C419 pad 2: /Audio Amplifier/MIC_IN -> Net-(C419-Pad2)
- C420 pad 1: NVCC_3V3 -> Net-(C420-Pad1)
- C420 pad 2: GND -> /Audio Amplifier/HPR
- C501 pad 1: +4V -> 4V_BST
- C502 pad 1: +4V -> 4V_BST
- C504 pad 2: /Radio Module, GPS and SIM/GSM_GND -> /Radio Module, GPS and SIM/GPS_GND
- C505 pad 2: /Radio Module, GPS and SIM/GPS_GND -> /Radio Module, GPS and SIM/GSM_GND
- C506 pad 1: /Radio Module, GPS and SIM/GSM_RF -> /Radio Module, GPS and SIM/GPS_RF
- C506 pad 2: /Radio Module, GPS and SIM/GSM_GND -> /Radio Module, GPS and SIM/GPS_GND
- C507 pad 1: /Radio Module, GPS and SIM/GPS_RF -> /Radio Module, GPS and SIM/GSM_RF
- C507 pad 2: /Radio Module, GPS and SIM/GPS_GND -> /Radio Module, GPS and SIM/GSM_GND
- C805 pad 1: Net-(C805-Pad1) -> /Controller/nRST
- C806 pad 1: Net-(C805-Pad1) -> Net-(C806-Pad1)
- C808 pad 1: Net-(C805-Pad1) -> Net-(C808-Pad1)
- C809 pad 1: /Buttons and LEDs/~ON -> NVCC_3V3
- C810 pad 1: SW2OUT -> NVCC_3V3
- C812 pad 1: VLDO_2V8 -> NVCC_3V3
- C813 pad 1: NVCC_1V8 -> NVCC_3V3
- C814 pad 1: Net-(C814-Pad1) -> NVCC_3V3
- C815 pad 1: NVCC_1V8 -> NVCC_3V3
- L202 pad 1: Net-(D205-Pad1) -> Net-(L202-Pad1)
- L202 pad 2: +BATT_LIPO -> 3V3
- P101 pad 2: /Controller/D- -> /Controller/USB_DN
- P101 pad 3: /Controller/D+ -> /Controller/USB_DP
- P101 pad 4: /Controller/USB_OTG_ID -> /Controller/USB_ID
- P107 pad 3: /Audio Amplifier/HPM -> Net-(P107-Pad3)
- P107 pad 5: /Audio Amplifier/HP_DETECT -> Net-(P107-Pad5)
- P301 pad 1: Net-(P301-Pad1) -> GND
- P301 pad 10: Net-(P301-Pad10) -> GND
- P301 pad 11: Net-(P301-Pad11) -> GND
- P301 pad 12: Net-(P301-Pad12) -> GND
- P301 pad 13: Net-(P301-Pad13) -> GND
- P301 pad 15: NVCC_3V3 -> GND
- P301 pad 19: Net-(P301-Pad19) -> GND
- P301 pad 20: Net-(P301-Pad20) -> GND
- P301 pad 21: Net-(P301-Pad21) -> GND
- P301 pad 22: Net-(P301-Pad22) -> GND
- P301 pad 23: Net-(P301-Pad23) -> GND
- P301 pad 24: Net-(P301-Pad24) -> GND
- P301 pad 28: Net-(P301-Pad28) -> GND
- P301 pad 30: Net-(P301-Pad30) -> GND
- P301 pad 31: GND -> NVCC_3V3
- P301 pad 32: /Display/VDD -> GND
- P301 pad 33: GND -> 18V_BST
- P301 pad 35: Net-(P301-Pad35) -> GND
- P301 pad 8: /Display/VDDIO -> NVCC_3V3
- P801 pad 2: Net-(P801-Pad2) -> /Controller/JTAG_TMS
- P801 pad 4: Net-(P801-Pad4) -> /Controller/JTAG_TCK
- P801 pad 6: Net-(P801-Pad6) -> /Controller/JTAG_TDO
- P801 pad 8: Net-(P801-Pad8) -> /Controller/JTAG_TDI
- R201 pad 1: /Controller/V_USB_BUS_ref -> /Controller/ADC1
- R202 pad 2: /Controller/V_USB_BUS_ref -> /Controller/ADC1
- R203 pad 2: /Controller/VDC_ref -> /Controller/ADC2
- R204 pad 1: /Controller/VDC_ref -> /Controller/ADC2
- R205 pad 1: Net-(D202-Pad1) -> Net-(R205-Pad1)
- R205 pad 2: Net-(C211-Pad1) -> +BATT_LIPO
- R206 pad 1: Net-(C211-Pad2) -> Net-(R206-Pad1)
- R206 pad 2: GND -> +BATT_LIPO
- R207 pad 2: /Controller/VBAT_ref -> /Controller/ADC3
- R208 pad 1: /Controller/VBAT_ref -> /Controller/ADC3
- R209 pad 1: GNDREF -> Net-(R209-Pad1)
- R209 pad 2: GND -> +BATT_LIPO
- R210 pad 1: Net-(C212-Pad1) -> Net-(R210-Pad1)
- R210 pad 2: GNDREF -> +BATT_LIPO
- R211 pad 1: Net-(C211-Pad1) -> GND
- R211 pad 2: /Controller/~CHARGING -> Net-(R205-Pad1)
- R212 pad 1: Net-(Q203-Pad1) -> GND
- R212 pad 2: Net-(C216-Pad1) -> Net-(R206-Pad1)
- R213 pad 1: Net-(Q202-Pad3) -> GND
- R213 pad 2: GNDREF -> Net-(R209-Pad1)
- R214 pad 1: Net-(R214-Pad1) -> GND
- R214 pad 2: Net-(C217-Pad1) -> Net-(R210-Pad1)
- R215 pad 1: +BATT_LIPO -> 3V3
- R215 pad 2: Net-(R214-Pad1) -> /Power and Battery/3V3_PG
- R305 pad 1: Net-(P301-Pad9) -> Net-(P301-Pad25)
- R305 pad 2: Net-(R305-Pad2) -> /Controller/LCD_RS
- R306 pad 1: Net-(P301-Pad10) -> Net-(P301-Pad26)
- R306 pad 2: /Controller/LCD_VSYNC -> GND
- R307 pad 1: Net-(P301-Pad11) -> Net-(R307-Pad1)
- R307 pad 2: /Controller/LCD_HSYNC -> /Controller/LCD_RESET
- R308 pad 1: Net-(P301-Pad12) -> Net-(P301-Pad17)
- R308 pad 2: /Controller/LCD_CLK -> GND
- R309 pad 1: Net-(P301-Pad13) -> Net-(R307-Pad1)
- R309 pad 2: /Controller/LCD_ENABLE -> GND
- R312 pad 1: Net-(P301-Pad18) -> Net-(P301-Pad16)
- R312 pad 2: /Display/DISPLAY_DATA7 -> GND
- R313 pad 1: Net-(P301-Pad19) -> Net-(P301-Pad26)
- R313 pad 2: /Display/DISPLAY_DATA6 -> GND
- R314 pad 1: Net-(P301-Pad20) -> Net-(P301-Pad25)
- R314 pad 2: /Display/DISPLAY_DATA5 -> GND
- R323 pad 1: Net-(P301-Pad30) -> Net-(P301-Pad29)
- R323 pad 2: /Controller/LCD_RESET -> Net-(R307-Pad1)
- R403 pad 1: VDD_SPK -> Net-(R403-Pad1)
- R403 pad 2: +4V -> NVCC_3V3
- R404 pad 1: /Audio Amplifier/HPR -> Net-(C418-Pad1)
- R404 pad 2: GNDA -> GND
- R405 pad 1: /Audio Amplifier/HPL -> Net-(C420-Pad1)
- R405 pad 2: GNDA -> GND
- R502 pad 2: +4V -> 4V_BST
- R503 pad 2: /Radio Module, GPS and SIM/GSM_RF -> /Radio Module, GPS and SIM/GPS_RF
- R504 pad 2: /Radio Module, GPS and SIM/GPS_RF -> /Radio Module, GPS and SIM/GSM_RF
- R505 pad 1: /Controller/GPS_TX -> /Radio Module, GPS and SIM/GPS_TX
- R701 pad 2: /Buttons and LEDs/~ON -> /Controller/SYS_WKUP
- R803 pad 1: Net-(R803-Pad1) -> Net-(C808-Pad1)
- R803 pad 2: GND -> NVCC_3V3
- R805 pad 2: Net-(P801-Pad8) -> /Controller/JTAG_TDI
- R806 pad 2: Net-(R806-Pad2) -> /Controller/JTAG_RST
- R807 pad 2: Net-(P801-Pad2) -> /Controller/JTAG_TMS
- SW701 pad 2: /Buttons and LEDs/~ON -> /Controller/SYS_WKUP
- TP201 pad 1: /Controller/V_USB_BUS_ref -> /Controller/ADC1
- TP202 pad 1: /Controller/VDC_ref -> /Controller/ADC2
- TP203 pad 1: /Controller/VBAT_ref -> /Controller/ADC3
- TP301 pad 1: Net-(TP301-Pad1) -> Net-(P301-Pad18)
- TP701 pad 1: /Buttons and LEDs/~ON -> /Controller/SYS_WKUP
- U202 pad 1: Net-(C212-Pad1) -> +BATT_LIPO
- U202 pad 2: GND -> Net-(L202-Pad1)
- U202 pad 3: /Controller/~CHARGING -> GND
- U202 pad 4: Net-(C217-Pad1) -> /Controller/NVCC_3V3_EN
- U202 pad 5: Net-(U202-Pad5) -> 3V3
- U202 pad 6: Net-(C211-Pad2) -> NVCC_3V3
- U202 pad 7: Net-(C211-Pad1) -> /Power and Battery/3V3_PG
- U202 pad 8: Net-(C214-Pad1) -> Net-(R210-Pad1)
- U301 pad 1: (no net) -> GND
- U301 pad 2: (no net) -> 4V_BST
- U301 pad 3: (no net) -> 4V_BST
- U504 pad 10: Net-(U501-Pad~) -> Net-(U501-Pad7)
- U504 pad 11: Net-(U501-Pad~) -> Net-(U501-Pad6)
- U504 pad 19: /Audio Amplifier/MIC_+ -> /Radio Module, GPS and SIM/MIC_+
- U504 pad 2: /Radio Module, GPS and SIM/GSM_GND -> /Radio Module, GPS and SIM/GPS_GND
- U504 pad 20: /Audio Amplifier/MIC_- -> /Radio Module, GPS and SIM/MIC_-
- U504 pad 30: Net-(U502-Pad~) -> Net-(U502-Pad7)
- U504 pad 31: Net-(U502-Pad~) -> Net-(U502-Pad6)
- U504 pad 32: Net-(U503-Pad~) -> Net-(U503-Pad7)
- U504 pad 33: Net-(U503-Pad~) -> Net-(U503-Pad6)
- U504 pad 34: /Radio Module, GPS and SIM/GPS_GND -> /Radio Module, GPS and SIM/GSM_GND
- U504 pad 36: /Radio Module, GPS and SIM/GPS_GND -> /Radio Module, GPS and SIM/GSM_GND
- U504 pad 41: +4V -> 4V_BST
- U504 pad 42: +4V -> 4V_BST
- U601 pad 1: /WiFi/BT Controller/SD2_BUS8 -> /Controller/WIFI_RESET
- U601 pad 12: Net-(U601-Pad12) -> /Controller/WIFI_BOOT0
- U601 pad 15: Net-(P601-Pad2) -> /Controller/USART6_RX
- U601 pad 16: Net-(P601-Pad1) -> /Controller/USART6_TX
- U601 pad 17: /WiFi/BT Controller/SD2_BUS1 -> Net-(U601-Pad17)
- U601 pad 18: /WiFi/BT Controller/SD2_BUS2 -> Net-(U601-Pad18)
- U601 pad 19: /WiFi/BT Controller/SD2_BUS4 -> Net-(U601-Pad19)
- U601 pad 20: /WiFi/BT Controller/SD2_BUS5 -> Net-(U601-Pad20)
- U601 pad 21: /WiFi/BT Controller/SD2_BUS3 -> Net-(U601-Pad21)
- U601 pad 22: /WiFi/BT Controller/SD2_BUS0 -> Net-(U601-Pad22)
- U601 pad 3: /WiFi/BT Controller/SD2_BUS6 -> /Controller/WIFI_CHPD
Routing:
- net /Controller/ADC2: track 0.00 -> 78.6 mm, vias 0 -> 2
- net /Controller/DDR3 RAM /SDCLK0_N: track 60.0 -> 0.00 mm, vias 3 -> 0
- net /Controller/DDR3 RAM /SDCLK0_P: track 59.6 -> 0.00 mm, vias 1 -> 0
- net /Controller/DDR3 RAM /DRAM_ADDR7: track 55.2 -> 0.00 mm, vias 3 -> 0
- net /Controller/ADC3: track 0.00 -> 47.3 mm, vias 0 -> 2
- net /Controller/USB_DN: track 0.00 -> 47.0 mm
- net /Controller/USB_DP: track 0.00 -> 46.8 mm
- net /Audio Amplifier/SPK_-: track 0.00 -> 38.9 mm
- net /Audio Amplifier/SPK_+: track 0.00 -> 37.6 mm
- net /Controller/DDR3 RAM /DRAM_ADDR13: track 37.5 -> 0.00 mm, vias 2 -> 0
- net NVCC_DRAM: track 33.7 -> 0.00 mm, vias 5 -> 0
- net GND: track 0.00 -> 22.2 mm, vias 194 -> 26
- net /Controller/DDR3 RAM /DRAM_ADDR8: track 21.4 -> 0.00 mm, vias 2 -> 0
- net /Controller/DDR3 RAM /DRAM_ADDR1: track 21.2 -> 0.00 mm, vias 2 -> 0
- net /Controller/DDR3 RAM /DRAM_ADDR11: track 20.2 -> 0.00 mm, vias 2 -> 0
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- added copper zone on B.Cu, net +5V
- added copper zone on B.Cu, net +BATT_LIPO
- added copper zone on In2.Cu, net +BATT_LIPO
- added copper zone on B.Cu, net GND
- added copper zone on B.Cu, net GNDREF
- added copper zone on B.Cu, net NVCC_1V8
- added copper zone on In2.Cu, net NVCC_1V8
- added copper zone on B.Cu, net NVCC_3V3
- added copper zone on F.Cu, net Net-(P101-Pad6)
- removed copper zone on BOT_GND, net GND
Other:
- copper layers 8 -> 4
- net class DDR_external removed
- net class Default: clearance 0.15 -> 0.2; via_drill 0.2 -> 0.3
- net class SmallPower removed
- rule trace_clearance: 0.15 -> 0.2
